File: reference/hardware/v0.3/Jag_Speedy/_autosave-Jag_Speedy.kicad_pcb (KiCad board)
At the start: 2 copper layers, 215 parts, among them IC1 MPX4250AP, IC10 SP720APP, IC11 VNLD5090-E, IC11 VNS3NV04DP-E, IC2 MPX4250AP, IC3 VNLD5090-E, IC3 VNS3NV04DP-E, IC4 VNLD5090-E, IC4 VNS3NV04DP-E, IC5 VNLD5090-E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

Commit message: Rationalise level shifting
Parts:
- moved J2 42.3 mm to (-40.6, 62.2)
- moved R39 32.4 mm to (-2.54, 29.2)
- moved R44 26.2 mm to (6.35, 35.6), turned to 180 degrees
- moved R38 25.4 mm to (3.81, 29.2), turned to 0 degrees
- moved R45 24.4 mm to (-2.54, 35.6), turned to 0 degrees
- moved IC5 11.4 mm to (0.00, 76.2)
- moved D9 10.2 mm to (-11.4, 57.1), turned to 180 degrees
- moved IC4 6.35 mm to (0.00, 61.0)
- moved IC3 1.27 mm to (0.00, 45.7)
Changed lines of the file:
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@@
   )
   (module Resistor_THT:R_Axial_DIN0207_L6.3mm_D2.5mm_P2.54mm_Vertical (layer F.Cu)
-    (at 16.51 50.8 270)
+    (at -2.54 35.56)
     (descr "Resistor, Axial_DIN0207 series, Axial, Vertical, pin pitch=2.54mm, 0.25W = 1/4W, length*diameter=6.3*2.5mm^2, http://cdn-reichelt.de/documents/datenblatt/B400/1_4W%23YAG.pdf")
     (tags "Resistor Axial_DIN0207 series Axial Vertical pin pitch 2.54mm 0.25W = 1/4W length 6.3mm diameter 2.5mm")
-    (fp_text reference R45 (at 1.27 -2.37 90) (layer F.SilkS)
+    (fp_text reference R45 (at 1.27 -2.37) (layer F.SilkS)
       (effects (font (size 1 1) (thickness 0.15)))
     )
-    (fp_text value 1k (at 1.27 2.37 90) (layer F.Fab)
+    (fp_text value 1k (at 1.27 2.37) (layer F.Fab)
       (effects (font (size 1 1) (thickness 0.15)))
     )
-    (fp_text user %R (at 1.27 -2.37 90) (layer F.Fab)
+    (fp_text user %R (at 1.27 -2.37) (layer F.Fab)
       (effects (font (size 1 1) (thickness 0.15)))
     )
@@
     (fp_line (start 3.59 1.5) (end 3.59 -1.5) (layer F.CrtYd) (width 0.05))
     (fp_line (start 3.59 -1.5) (end -1.5 -1.5) (layer F.CrtYd) (width 0.05))
-    (pad 2 thru_hole oval (at 2.54 0 270) (size 1.6 1.6) (drill 0.8) (layers *.Cu *.Mask)
+    (pad 2 thru_hole oval (at 2.54 0) (size 1.6 1.6) (drill 0.8) (layers *.Cu *.Mask)
       (net 54 "Net-(IC3-Pad3)"))
-    (pad 1 thru_hole circle (at 0 0 270) (size 1.6 1.6) (drill 0.8) (layers *.Cu *.Mask)
+    (pad 1 thru_hole circle (at 0 0) (size 1.6 1.6) (drill 0.8) (layers *.Cu *.Mask)
       (net 129 Inj02-CPU-D09))
     (model ${KISYS3DMOD}/Resistor_THT.3dshapes/R_Axial_DIN0207_L6.3mm_D2.5mm_P2.54mm_Vertical.wrl
@@
   )
   (module Resistor_THT:R_Axial_DIN0207_L6.3mm_D2.5mm_P2.54mm_Vertical (layer F.Cu)
-    (at 16.51 59.69)
+    (at 6.35 35.56 180)
     (descr "Resistor, Axial_DIN0207 series, Axial, Vertical, pin pitch=2.54mm, 0.25W = 1/4W, length*diameter=6.3*2.5mm^2, http://cdn-reichelt.de/documents/datenblatt/B400/1_4W%23YAG.pdf")
     (tags "Resistor Axial_DIN0207 series Axial Vertical pin pitch 2.54mm 0.25W = 1/4W length 6.3mm diameter 2.5mm")
@@
     (fp_line (start 3.59 1.5) (end 3.59 -1.5) (layer F.CrtYd) (width 0.05))
     (fp_line (start 3.59 -1.5) (end -1.5 -1.5) (layer F.CrtYd) (width 0.05))
-    (pad 2 thru_hole oval (at 2.54 0) (size 1.6 1.6) (drill 0.8) (layers *.Cu *.Mask)
+    (pad 2 thru_hole oval (at 2.54 0 180) (size 1.6 1.6) (drill 0.8) (layers *.Cu *.Mask)
       (net 56 "Net-(IC3-Pad1)"))
-    (pad 1 thru_hole circle (at 0 0) (size 1.6 1.6) (drill 0.8) (layers *.Cu *.Mask)
+    (pad 1 thru_hole circle (at 0 0 180) (size 1.6 1.6) (drill 0.8) (layers *.Cu *.Mask)
       (net 128 Inj01-CPU-D08))
     (model ${KISYS3DMOD}/Resistor_THT.3dshapes/R_Axial_DIN0207_L6.3mm_D2.5mm_P2.54mm_Vertical.wrl
@@
   )
   (module Resistor_THT:R_Axial_DIN0207_L6.3mm_D2.5mm_P2.54mm_Vertical (layer F.Cu)
-    (at 21.59 50.8)
+    (at -2.54 29.21)
     (descr "Resistor, Axial_DIN0207 series, Axial, Vertical, pin pitch=2.54mm, 0.25W = 1/4W, length*diameter=6.3*2.5mm^2, http://cdn-reichelt.de/documents/datenblatt/B400/1_4W%23YAG.pdf")
     (tags "Resistor Axial_DIN0207 series Axial Vertical pin pitch 2.54mm 0.25W = 1/4W length 6.3mm diameter 2.5mm")
@@
   )
   (module Resistor_THT:R_Axial_DIN0207_L6.3mm_D2.5mm_P2.54mm_Vertical (layer F.Cu)
-    (at 24.13 44.45 180)
+    (at 3.81 29.21)
     (descr "Resistor, Axial_DIN0207 series, Axial, Vertical, pin pitch=2.54mm, 0.25W = 1/4W, length*diameter=6.3*2.5mm^2, http://cdn-reichelt.de/documents/datenblatt/B400/1_4W%23YAG.pdf")
     (tags "Resistor Axial_DIN0207 series Axial Vertical pin pitch 2.54mm 0.25W = 1/4W length 6.3mm diameter 2.5mm")
@@
     (fp_line (start 3.59 1.5) (end 3.59 -1.5) (layer F.CrtYd) (width 0.05))
     (fp_line (start 3.59 -1.5) (end -1.5 -1.5) (layer F.CrtYd) (width 0.05))
-    (pad 2 thru_hole oval (at 2.54 0 180) (size 1.6 1.6) (drill 0.8) (layers *.Cu *.Mask)
+    (pad 2 thru_hole oval (at 2.54 0) (size 1.6 1.6) (drill 0.8) (layers *.Cu *.Mask)
       (net 128 Inj01-CPU-D08))
-    (pad 1 thru_hole circle (at 0 0 180) (size 1.6 1.6) (drill 0.8) (layers *.Cu *.Mask)
+    (pad 1 thru_hole circle (at 0 0) (size 1.6 1.6) (drill 0.8) (layers *.Cu *.Mask)
       (net 17 PowerGnd))
     (model ${KISYS3DMOD}/Resistor_THT.3dshapes/R_Axial_DIN0207_L6.3mm_D2.5mm_P2.54mm_Vertical.wrl
@@
   )
   (module Connector_PinHeader_1.00mm:PinHeader_2x06_P1.00mm_Horizontal (layer F.Cu)
-    (at -17.78 97.79 180)
+    (at -40.64 62.23 180)
     (descr "Through hole angled pin header, 2x06, 1.00mm pitch, 2.0mm pin length, double rows")
     (tags "Through hole angled pin header THT 2x06 1.00mm double row")
@@
   )
   (module Package_SO:SO-8_5.3x6.2mm_P1.27mm (layer F.Cu)
-    (at 0 64.77 270)
+    (at 0 76.2 270)
     (descr "SO, 8 Pin (https://www.ti.com/lit/ml/msop001a/msop001a.pdf), generated with kicad-footprint-generator ipc_gullwing_generator.py")
     (tags "SO SO")
@@
   )
   (module Package_SO:SO-8_5.3x6.2mm_P1.27mm (layer F.Cu)
-    (at 0 54.61 270)
+    (at 0 60.96 270)
     (descr "SO, 8 Pin (https://www.ti.com/lit/ml/msop001a/msop001a.pdf), generated with kicad-footprint-generator ipc_gullwing_generator.py")
     (tags "SO SO")
@@
   )
   (module Package_SO:SO-8_5.3x6.2mm_P1.27mm (layer F.Cu)
-    (at 0 44.45 270)
+    (at 0 45.72 270)
     (descr "SO, 8 Pin (https://www.ti.com/lit/ml/msop001a/msop001a.pdf), generated with kicad-footprint-generator ipc_gullwing_generator.py")
     (tags "SO SO")
@@
   )
   (module Diode_THT:D_DO-41_SOD81_P10.16mm_Horizontal (layer F.Cu)
-    (at -21.59 57.15)
+    (at -11.43 57.15 180)
     (descr "Diode, DO-41_SOD81 series, Axial, Horizontal, pin pitch=10.16mm, , length*diameter=5.2*2.7mm^2, , http://www.diodes.com/_files/packages/DO-41%20(Plastic).pdf")
     (tags "Diode DO-41_SOD81 series Axial Horizontal pin pitch 10.16mm  length 5.2mm diameter 2.7mm")
@@
     (fp_line (start 11.51 1.6) (end 11.51 -1.6) (layer F.CrtYd) (width 0.05))
     (fp_line (start 11.51 -1.6) (end -1.35 -1.6) (layer F.CrtYd) (width 0.05))
-    (pad 2 thru_hole oval (at 10.16 0) (size 2.2 2.2) (drill 1.1) (layers *.Cu *.Mask)
+    (pad 2 thru_hole oval (at 10.16 0 180) (size 2.2 2.2) (drill 1.1) (layers *.Cu *.Mask)
       (net 25 "Net-(D3-Pad1)"))
-    (pad 1 thru_hole rect (at 0 0) (size 2.2 2.2) (drill 1.1) (layers *.Cu *.Mask)
+    (pad 1 thru_hole rect (at 0 0 180) (size 2.2 2.2) (drill 1.1) (layers *.Cu *.Mask)
       (net 34 Inj03-OUT))
     (model ${KISYS3DMOD}/Diode_THT.3dshapes/D_DO-41_SOD81_P10.16mm_Horizontal.wrl

Commit message: Schematic tidyup
Parts:
- added IC12: SP720APP, Package_DIP:DIP-16_W7.62mm, F.Cu at (151.0, 114.6)
- added R1: 180k, Resistor_THT:R_Axial_DIN0207_L6.3mm_D2.5mm_P2.54mm_Vertical, F.Cu at (174.0, 114.6)
- added R2: 180k, Resistor_THT:R_Axial_DIN0207_L6.3mm_D2.5mm_P2.54mm_Vertical, F.Cu at (180.1, 114.6)
- added R3: 330k, Resistor_THT:R_Axial_DIN0207_L6.3mm_D2.5mm_P2.54mm_Vertical, F.Cu at (174.0, 118.6)
- added R4: 330k, Resistor_THT:R_Axial_DIN0207_L6.3mm_D2.5mm_P2.54mm_Vertical, F.Cu at (180.1, 118.6)
- added R5: 330k, Resistor_THT:R_Axial_DIN0207_L6.3mm_D2.5mm_P2.54mm_Vertical, F.Cu at (174.0, 122.7)
- added R6: 330k, Resistor_THT:R_Axial_DIN0207_L6.3mm_D2.5mm_P2.54mm_Vertical, F.Cu at (186.3, 114.6)
- added R7: 180k, Resistor_THT:R_Axial_DIN0207_L6.3mm_D2.5mm_P2.54mm_Vertical, F.Cu at (174.0, 126.7)
- added R8: 180k, Resistor_THT:R_Axial_DIN0207_L6.3mm_D2.5mm_P2.54mm_Vertical, F.Cu at (180.1, 122.7)
- added U1: LMV324, Package_DIP:DIP-14_W7.62mm_Socket, F.Cu at (162.3, 114.7)
Connections:
- IC10 pad 10: ADCClamp09 -> Net-(IC10-Pad10)
- IC10 pad 11: ADCClamp10 -> Net-(IC10-Pad11)
- IC10 pad 12: ADCClamp11 -> Net-(IC10-Pad12)
- IC10 pad 5: ADCClamp05 -> Net-(IC10-Pad5)
- R23 pad 1: 5V -> 3V3
- R24 pad 1: 5V -> 3V3
- R25 pad 1: 5V -> 3V3
- R26 pad 1: 5V -> 3V3
- U3 pad 41: CPU-A0 -> ADCClamp08
- U3 pad 42: CLT-Signal-3.3V -> ADCClamp09
- U3 pad 45: BRV-Signal-3.3V -> ADCClamp05
- U3 pad 56: CPU-A10 -> ADCClamp10
- U3 pad 57: CPU-A11 -> ADCClamp11
