File: reference/hardware/v0.3/Jag_Speedy/connectors.sch (KiCad schematic (older format))
At the start: 8 parts, among them J1 Inputs, J2 Ouputs01, J3 Outputs02, J4 Power, J5 Bluetooth, J7 Canbus, U5 SN65HVD230

Commit message: Rationalise level shifting
Parts:
- R92: footprint (none) -> Resistor_THT:R_Axial_DIN0207_L6.3mm_D2.5mm_P2.54mm_Vertical
Connections:
- net VVT-OUT renamed CCPump-OUT
Other:
- note added: "Inputs"
- note added: "Outputs"
- note added: "Pin Mapping"
Changed lines of the file:
@@
 BoostPWM-OUT
 Text GLabel 2200 4900 0    50   Input ~ 0
-VVT-OUT
+CCPump-OUT
 Wire Wire Line
 	2200 5500 2400 5500
@@
 Text GLabel 7300 2350 2    50   Input ~ 0
 CPU-D12
-Text GLabel 7300 3700 2    50   Input ~ 0
+Text GLabel 7300 3800 2    50   Input ~ 0
 CPU-D07
 Text GLabel 7000 2350 0    50   Output ~ 0
@@
 Wire Wire Line
 	7300 2500 7000 2500
-Text GLabel 7000 2650 0    50   Output ~ 0
+Text GLabel 7000 2700 0    50   Output ~ 0
 Ign01-Trigger
-Text GLabel 7000 2800 0    50   Output ~ 0
+Text GLabel 7000 2850 0    50   Output ~ 0
 Ign02-Trigger
-Text GLabel 7000 2950 0    50   Output ~ 0
+Text GLabel 7000 3000 0    50   Output ~ 0
 Ign03-Trigger
-Text GLabel 7000 3100 0    50   Output ~ 0
+Text GLabel 7000 3150 0    50   Output ~ 0
 Ign04-Trigger
-Text GLabel 7000 3250 0    50   Output ~ 0
+Text GLabel 7000 3300 0    50   Output ~ 0
 Ign05-Trigger
-Text GLabel 7000 3400 0    50   Output ~ 0
+Text GLabel 7000 3450 0    50   Output ~ 0
 Ign06-Trigger
-Text GLabel 7300 2650 2    50   Input ~ 0
+Text GLabel 7300 2700 2    50   Input ~ 0
 CPU-D39
-Text GLabel 7300 2800 2    50   Input ~ 0
+Text GLabel 7300 2850 2    50   Input ~ 0
 CPU-D38
-Text GLabel 7300 2950 2    50   Input ~ 0
+Text GLabel 7300 3000 2    50   Input ~ 0
 CPU-D31
-Text GLabel 7300 3100 2    50   Input ~ 0
+Text GLabel 7300 3150 2    50   Input ~ 0
 CPU-D21
-Text GLabel 7300 3250 2    50   Input ~ 0
+Text GLabel 7300 3300 2    50   Input ~ 0
 CPU-D32
-Text GLabel 7300 3400 2    50   Input ~ 0
+Text GLabel 7300 3450 2    50   Input ~ 0
 CPU-D35
 Wire Wire Line
-	7000 2650 7300 2650
-Wire Wire Line
-	7300 2800 7000 2800
-Wire Wire Line
-	7000 2950 7300 2950
-Wire Wire Line
-	7300 3100 7000 3100
-Wire Wire Line
-	7000 3250 7300 3250
-Wire Wire Line
-	7300 3400 7000 3400
-Text GLabel 7000 3550 0    50   Output ~ 0
+	7000 2700 7300 2700
+Wire Wire Line
+	7300 2850 7000 2850
+Wire Wire Line
+	7000 3000 7300 3000
+Wire Wire Line
+	7300 3150 7000 3150
+Wire Wire Line
+	7000 3300 7300 3300
+Wire Wire Line
+	7300 3450 7000 3450
+Text GLabel 7000 3650 0    50   Output ~ 0
 IdlePWM-Signal
-Text GLabel 7000 3850 0    50   Output ~ 0
+Text GLabel 7000 3950 0    50   Output ~ 0
 TachoOut-Signal
-Text GLabel 7000 4000 0    50   Output ~ 0
+Text GLabel 7000 4100 0    50   Output ~ 0
 Fan-Signal
-Text GLabel 7000 4150 0    50   Output ~ 0
+Text GLabel 7000 4250 0    50   Output ~ 0
 FuelPump-Signal
-Text GLabel 7300 3550 2    50   Input ~ 0
+Text GLabel 7300 3650 2    50   Input ~ 0
 CPU-D05
 Text GLabel 7300 2500 2    50   Input ~ 0
 CPU-D13
-Text GLabel 7300 3850 2    50   Input ~ 0
+Text GLabel 7300 3950 2    50   Input ~ 0
 CPU-D28
-Text GLabel 7300 4000 2    50   Input ~ 0
+Text GLabel 7300 4100 2    50   Input ~ 0
 CPU-D27
-Text GLabel 7300 4150 2    50   Input ~ 0
+Text GLabel 7300 4250 2    50   Input ~ 0
 CPU-D37
-Text GLabel 7000 3700 0    50   Output ~ 0
+Text GLabel 7000 3800 0    50   Output ~ 0
 BoostPWM-Signal
-Text GLabel 7000 4300 0    50   Output ~ 0
+Text GLabel 7000 4400 0    50   Output ~ 0
 Idle02-Signal
-Text GLabel 7300 4300 2    50   Input ~ 0
+Text GLabel 7300 4400 2    50   Input ~ 0
 CPU-D06
-Text GLabel 7000 4450 0    50   Output ~ 0
-VVT-Signal
-Wire Wire Line
-	7000 3550 7300 3550
-Wire Wire Line
-	7300 3700 7000 3700
-Wire Wire Line
-	7000 3850 7300 3850
-Wire Wire Line
-	7300 4000 7000 4000
-Wire Wire Line
-	7000 4150 7300 4150
-Wire Wire Line
-	7300 4300 7000 4300
-Text GLabel 7300 4450 2    50   Input ~ 0
+Text GLabel 7000 4550 0    50   Output ~ 0
+CCPump-Signal
+Wire Wire Line
+	7000 3650 7300 3650
+Wire Wire Line
+	7300 3800 7000 3800
+Wire Wire Line
+	7000 3950 7300 3950
+Wire Wire Line
+	7300 4100 7000 4100
+Wire Wire Line
+	7000 4250 7300 4250
+Wire Wire Line
+	7300 4400 7000 4400
+Text GLabel 7300 4550 2    50   Input ~ 0
 CPU-D29
 Wire Wire Line
-	7300 4450 7000 4450
+	7300 4550 7000 4550
 Text GLabel 8800 1900 0    50   Input ~ 0
 O2-Signal-3.3V
@@
 CPU-A2
 Text GLabel 8800 2200 0    50   Input ~ 0
-BRV-Signal-3.3V
+BRV-Signal-3V3
 Text GLabel 9250 2200 2    50   Output ~ 0
 CPU-A4
@@
 CPU-A5
 Text GLabel 8800 2650 0    50   Input ~ 0
-CLT-Signal-3.3V
+CLT-Signal-3V3
 Text GLabel 9250 2650 2    50   Output ~ 0
 CPU-A1
 Text GLabel 8800 2800 0    50   Input ~ 0
-FPress-Signal-3.3V
+FPress-Signal-3V3
 Text GLabel 9250 2800 2    50   Output ~ 0
 CPU-A10
 Text GLabel 8800 2950 0    50   Input ~ 0
-OPress-Signal-3.3V
+OPress-Signal-3V3
 Text GLabel 9250 2950 2    50   Output ~ 0
 CPU-A11
-Text GLabel 8800 3350 0    50   Input ~ 0
+Text GLabel 8800 3300 0    50   Input ~ 0
 FlexFuel-Signal
-Text GLabel 8800 3200 0    50   Input ~ 0
+Text GLabel 8800 3150 0    50   Input ~ 0
 ClutchIn-Signal
-Text GLabel 9250 3200 2    50   Output ~ 0
+Text GLabel 9250 3150 2    50   Output ~ 0
 CPU-D24
-Text GLabel 9250 3350 2    50   Output ~ 0
+Text GLabel 9250 3300 2    50   Output ~ 0
 CPU-D25
 Wire Wire Line
@@
 	9250 2950 8800 2950
 Wire Wire Line
-	8800 3200 9250 3200
-Wire Wire Line
-	9250 3350 8800 3350
-Text GLabel 8800 4000 0    50   Input ~ 0
-Spare-Signal-3.3V-02
-Text GLabel 8800 4150 0    50   Input ~ 0
-Spare-Signal-3.3V-03
-Text GLabel 8800 3850 0    50   Input ~ 0
-Spare-Signal-3.3V-01
+	8800 3150 9250 3150
+Wire Wire Line
+	9250 3300 8800 3300
 Text GLabel 8800 1750 0    50   Input ~ 0
-IAT-Signal-3.3V
+IAT-Signal-3V3
 Text GLabel 9250 1750 2    50   Output ~ 0
 CPU-A0
 Wire Wire Line
 	8800 1750 9250 1750
-Text GLabel 8800 3550 0    50   Input ~ 0
+Text GLabel 8800 3500 0    50   Input ~ 0
 Crank-Signal
-Text GLabel 8800 3700 0    50   Input ~ 0
+Text GLabel 8800 3650 0    50   Input ~ 0
 Cam-Signal
-Text GLabel 9250 3700 2    50   Output ~ 0
+Text GLabel 9250 3650 2    50   Output ~ 0
 CPU-D36
-Text GLabel 9250 3550 2    50   Output ~ 0
+Text GLabel 9250 3500 2    50   Output ~ 0
 CPU-D23
 Wire Wire Line
-	8800 3700 9250 3700
-Wire Wire Line
-	9250 3550 8800 3550
+	8800 3650 9250 3650
+Wire Wire Line
+	9250 3500 8800 3500
 $Comp
 L Interface_CAN_LIN:SN65HVD230 U?
@@
 F 0 "R92" V 4407 5150 50  0000 C CNN
 F 1 "10K" V 4316 5150 50  0000 C CNN
-F 2 "" V 4130 5150 50  0001 C CNN
+F 2 "Resistor_THT:R_Axial_DIN0207_L6.3mm_D2.5mm_P2.54mm_Vertical" V 4130 5150 50  0001 C CNN
 F 3 "~" H 4200 5150 50  0001 C CNN
 	1    4200 5150
@@
 	5100 4600 4850 4600
 NoConn ~ 4050 4700
+Text Notes 7350 1200 0    157  ~ 0
+Pin Mapping
+Text Notes 6650 1550 0    157  ~ 0
+Outputs
+Text Notes 8500 1550 0    157  ~ 0
+Inputs
 $EndSCHEMATC

Commit message: Schematic tidyup
Parts:
- J2: footprint Connector_PinHeader_1.00mm:PinHeader_2x06_P1.00mm_Horizontal -> Connector_PinHeader_1.00mm:PinHeader_2x07_P1.00mm_Horizontal; symbol Connector_Generic:Conn_01x12 -> Connector_Generic:Conn_01x14
Connections:
- net 3V3: now also J1.1 (Pin_1), J1.12 (Pin_12)
- net 5V: no longer J1.12 (Pin_12)
- net GND: now also J2.1 (Pin_1), J2.14 (Pin_14), J3.10 (Pin_10), J3.3 (Pin_3), J3.9 (Pin_9)
- net Ign01-OUT: now also J2.8 (Pin_8); no longer J2.7 (Pin_7)
- net Ign02-OUT: now also J2.9 (Pin_9); no longer J2.8 (Pin_8)
- net Ign03-OUT: now also J2.10 (Pin_10); no longer J2.9 (Pin_9)
- net Ign04-OUT: now also J2.11 (Pin_11); no longer J2.10 (Pin_10)
- net Ign05-OUT: now also J2.12 (Pin_12); no longer J2.11 (Pin_11)
- net Ign06-OUT: now also J2.13 (Pin_13); no longer J2.12 (Pin_12)
- net Inj01-OUT: now also J2.2 (Pin_2); no longer J2.1 (Pin_1)
- net Inj02-OUT: now also J2.3 (Pin_3); no longer J2.2 (Pin_2)
- net Inj03-OUT: now also J2.4 (Pin_4); no longer J2.3 (Pin_3)
- net Inj04-OUT: now also J2.5 (Pin_5); no longer J2.4 (Pin_4)
- net Inj05-OUT: now also J2.6 (Pin_6); no longer J2.5 (Pin_5)
- net Inj06-OUT: now also J2.7 (Pin_7); no longer J2.6 (Pin_6)
- no-connect marks 7 -> 3
Other:
- moved on the sheet: J3
Changed lines of the file:
@@
 	1    0    0    -1
 $EndComp
-Text GLabel 2250 1200 0    50   Output ~ 0
+Text GLabel 2250 1200 0    50   Input ~ 0
 TPSSensor
-Text GLabel 2250 1400 0    50   Output ~ 0
+Text GLabel 2250 1400 0    50   Input ~ 0
 IATSensor
-Text GLabel 2250 1600 0    50   Output ~ 0
+Text GLabel 2250 1600 0    50   Input ~ 0
 CLTSensor
-Text GLabel 2250 1800 0    50   Output ~ 0
+Text GLabel 2250 1800 0    50   Input ~ 0
 O2Sensor
-Text GLabel 2250 2200 0    50   Output ~ 0
+Text GLabel 2250 2200 0    50   Input ~ 0
 CrankSensor+
 $Comp
-L Connector_Generic:Conn_01x12 J2
+L Connector_Generic:Conn_01x14 J2
 U 1 1 5EF06693
-P 2600 3950
-F 0 "J2" H 2680 3942 50  0000 L CNN
-F 1 "Ouputs01" H 2680 3851 50  0000 L CNN
-F 2 "Connector_PinHeader_1.00mm:PinHeader_2x06_P1.00mm_Horizontal" H 2600 3950 50  0001 C CNN
-F 3 "~" H 2600 3950 50  0001 C CNN
-	1    2600 3950
+P 2600 4150
+F 0 "J2" H 2680 4142 50  0000 L CNN
+F 1 "Ouputs01" H 2680 4051 50  0000 L CNN
+F 2 "Connector_PinHeader_1.00mm:PinHeader_2x07_P1.00mm_Horizontal" H 2600 4150 50  0001 C CNN
+F 3 "~" H 2600 4150 50  0001 C CNN
+	1    2600 4150
 	1    0    0    -1
 $EndComp
-Text GLabel 2150 3450 0    50   Input ~ 0
+Text GLabel 2150 3650 0    50   Output ~ 0
 Inj01-OUT
-Text GLabel 2150 3550 0    50   Input ~ 0
+Text GLabel 2150 3750 0    50   Output ~ 0
 Inj02-OUT
-Text GLabel 2150 3650 0    50   Input ~ 0
+Text GLabel 2150 3850 0    50   Output ~ 0
 Inj03-OUT
-Text GLabel 2150 3750 0    50   Input ~ 0
+Text GLabel 2150 3950 0    50   Output ~ 0
 Inj04-OUT
-Text GLabel 2150 3850 0    50   Input ~ 0
+Text GLabel 2150 4050 0    50   Output ~ 0
 Inj05-OUT
-Text GLabel 2150 3950 0    50   Input ~ 0
+Text GLabel 2150 4150 0    50   Output ~ 0
 Inj06-OUT
-Text GLabel 2150 4050 0    50   Input ~ 0
+Text GLabel 2150 4250 0    50   Output ~ 0
 Ign01-OUT
-Text GLabel 2150 4150 0    50   Input ~ 0
+Text GLabel 2150 4350 0    50   Output ~ 0
 Ign02-OUT
-Text GLabel 2150 4250 0    50   Input ~ 0
+Text GLabel 2150 4450 0    50   Output ~ 0
 Ign03-OUT
-Text GLabel 2150 4350 0    50   Input ~ 0
+Text GLabel 2150 4550 0    50   Output ~ 0
 Ign04-OUT
-Text GLabel 2150 4450 0    50   Input ~ 0
+Text GLabel 2150 4650 0    50   Output ~ 0
 Ign05-OUT
-Text GLabel 2150 4550 0    50   Input ~ 0
+Text GLabel 2150 4750 0    50   Output ~ 0
 Ign06-OUT
 $Comp
@@
 	-1   0    0    1
 $EndComp
-Text GLabel 2250 2400 0    50   Output ~ 0
+Text GLabel 2250 2400 0    50   Input ~ 0
 CamSensor+
-Text GLabel 2250 2700 0    50   Output ~ 0
+Text GLabel 2250 2700 0    50   Input ~ 0
 FuelPressureSensor
-Text GLabel 2250 2900 0    50   Output ~ 0
+Text GLabel 2250 2900 0    50   Input ~ 0
 OilPressureSensor
 $Comp
 L Connector_Generic:Conn_01x10 J3
 U 1 1 5EF09634
-P 2600 5200
-F 0 "J3" H 2680 5192 50  0000 L CNN
-F 1 "Outputs02" H 2680 5101 50  0000 L CNN
-F 2 "Connector_PinHeader_1.00mm:PinHeader_2x05_P1.00mm_Horizontal" H 2600 5200 50  0001 C CNN
-F 3 "~" H 2600 5200 50  0001 C CNN
-	1    2600 5200
+P 2600 5600
+F 0 "J3" H 2680 5592 50  0000 L CNN
+F 1 "Outputs02" H 2680 5501 50  0000 L CNN
+F 2 "Connector_PinHeader_1.00mm:PinHeader_2x05_P1.00mm_Horizontal" H 2600 5600 50  0001 C CNN
+F 3 "~" H 2600 5600 50  0001 C CNN
+	1    2600 5600
 	1    0    0    -1
 $EndComp
-Text GLabel 2200 5100 0    50   Input ~ 0
+Text GLabel 2200 5500 0    50   Output ~ 0
 FuelPump-OUT
-Text GLabel 2200 5200 0    50   Input ~ 0
+Text GLabel 2200 5600 0    50   Output ~ 0
 Fan-OUT
-Text GLabel 2200 5300 0    50   Input ~ 0
+Text GLabel 2200 5700 0    50   Output ~ 0
 IdlePWM-OUT
-Text GLabel 2250 2000 0    50   Input ~ 0
-5V
-Text GLabel 2250 2600 0    50   Input ~ 0
+Text GLabel 2250 2000 0    50   Output ~ 0
+3V3
+Text GLabel 2250 2600 0    50   Output ~ 0
 5V
 Wire Wire Line
@@
 SignalGnd
 Wire Wire Line
-	2150 3450 2400 3450
-Wire Wire Line
-	2400 3550 2150 3550
-Wire Wire Line
 	2150 3650 2400 3650
 Wire Wire Line
@@
 	2400 4550 2150 4550
 Wire Wire Line
-	2200 5100 2400 5100
-Wire Wire Line
-	2400 5200 2200 5200
-Wire Wire Line
-	2200 5300 2400 5300
+	2150 4650 2400 4650
+Wire Wire Line
+	2400 4750 2150 4750
+Wire Wire Line
+	2200 5500 2400 5500
+Wire Wire Line
+	2400 5600 2200 5600
+Wire Wire Line
+	2200 5700 2400 5700
 Text GLabel 4800 3250 2    50   Input ~ 0
 SignalGnd
@@
 Wire Wire Line
 	4800 3050 4300 3050
-Text GLabel 2250 2300 0    50   Output ~ 0
+Text GLabel 2250 2300 0    50   Input ~ 0
 CrankSensor-
-Text GLabel 2250 2500 0    50   Output ~ 0
+Text GLabel 2250 2500 0    50   Input ~ 0
 CamSensor-
 Wire Wire Line
@@
 Wire Wire Line
 	4800 2150 4300 2150
-Text GLabel 2250 1000 0    50   Output ~ 0
+Text GLabel 2250 1000 0    50   Input ~ 0
 FlexFuelSensor
-Text GLabel 2250 3100 0    50   Output ~ 0
+Text GLabel 2250 3100 0    50   Input ~ 0
 ClutchSwitch
 Wire Wire Line
@@
 	1400 3200 1400 3000
 Connection ~ 1400 3000
-Text GLabel 2200 5500 0    50   Input ~ 0
+Text GLabel 2200 5900 0    50   Output ~ 0
 Tacho-OUT
-Text GLabel 2200 4800 0    50   Input ~ 0
+Text GLabel 2200 5200 0    50   Output ~ 0
 BoostPWM-OUT
-Text GLabel 2200 4900 0    50   Input ~ 0
+Text GLabel 2200 5300 0    50   Output ~ 0
 CCPump-OUT
 Wire Wire Line
-	2200 5500 2400 5500
-Wire Wire Line
-	2200 4800 2400 4800
-Wire Wire Line
-	2200 4900 2400 4900
-Text GLabel 2200 5400 0    50   Input ~ 0
+	2200 5900 2400 5900
+Wire Wire Line
+	2200 5200 2400 5200
+Wire Wire Line
+	2200 5300 2400 5300
+Text GLabel 2200 5800 0    50   Output ~ 0
 Idle02-OUT
 Wire Wire Line
-	2200 5400 2400 5400
+	2200 5800 2400 5800
 Wire Wire Line
 	4300 3150 4800 3150
@@
 Wire Wire Line
 	4900 1100 4900 1300
-NoConn ~ 2400 900
 NoConn ~ 4300 2750
 NoConn ~ 4300 2850
-NoConn ~ 2400 5700
-NoConn ~ 2400 5600
-NoConn ~ 2400 5000
 Wire Wire Line
 	4300 1750 4800 1750
@@
 U 1 1 5F25E793
 P 5300 4600
-F 0 "J7" H 5218 4075 50  0000 C CNN
-F 1 "Canbus" H 5218 4166 50  0000 C CNN
+F 0 "J7" H 5300 4250 50  0000 C CNN
+F 1 "Canbus" H 5300 4350 50  0000 C CNN
 F 2 "Connector_PinHeader_1.00mm:PinHeader_1x06_P1.00mm_Horizontal" H 5300 4600 50  0001 C CNN
 F 3 "~" H 5300 4600 50  0001 C CNN
@@
 Text Notes 8500 1550 0    157  ~ 0
 Inputs
+Text GLabel 2250 900  0    50   Output ~ 0
+3V3
+Wire Wire Line
+	2400 900  2250 900
+Text GLabel 2200 5400 0    50   Input ~ 0
+PowerGnd
+Wire Wire Line
+	2200 6100 2400 6100
+Wire Wire Line
+	2400 6000 2200 6000
+Wire Wire Line
+	2200 5400 2400 5400
+Text GLabel 2150 3550 0    50   Input ~ 0
+PowerGnd
+Wire Wire Line
+	2150 3550 2400 3550
+Text GLabel 2150 4850 0    50   Input ~ 0
+PowerGnd
+Wire Wire Line
+	2400 4850 2150 4850
+Text GLabel 2200 6100 0    50   Input ~ 0
+PowerGnd
+Text GLabel 2200 6000 0    50   Input ~ 0
+PowerGnd
 $EndSCHEMATC

Commit message: SMD Update
Parts:
- R92: footprint Resistor_THT:R_Axial_DIN0207_L6.3mm_D2.5mm_P2.54mm_Vertical -> Resistor_SMD:R_0805_2012Metric
Changed lines of the file:
@@
 F 0 "R92" V 4407 5150 50  0000 C CNN
 F 1 "10K" V 4316 5150 50  0000 C CNN
-F 2 "Resistor_THT:R_Axial_DIN0207_L6.3mm_D2.5mm_P2.54mm_Vertical" V 4130 5150 50  0001 C CNN
+F 2 "Resistor_SMD:R_0805_2012Metric" V 4130 5150 50  0001 C CNN
 F 3 "~" H 4200 5150 50  0001 C CNN
 	1    4200 5150
