File: reference/hardware/v0.3/Jag_Speedy/outputs.sch (KiCad schematic (older format))
At the start: 8 parts, among them IC11 VNLD5090-E, Q1 SSM3K357R,LF, Q2 SSM3K357R,LF, Q3 SSM3K357R,LF

Commit message: Schematic pin mapping
Connections:
- net BoostPWM-OUT: now also IC11.6 (DRAIN2); no longer IC11.8 (DRAIN1)
- net IdlePWM-OUT: now also IC11.8 (DRAIN1); no longer IC11.6 (DRAIN2)
- net BoostPWM-CPU-A21 renamed BoostPWM-Signal
- net Fan-CPU-D27 renamed Fan-Signal
- net FuelPump-CPU-D37 renamed FuelPump-Signal
- net IdlePWM-CPU-D05 renamed IdlePWM-Signal
- net TachoOut-CPU-D28 renamed TachoOut-Signal
Changed lines of the file:
@@
 PowerGnd
 Text GLabel 1450 4050 0    50   Input ~ 0
-FuelPump-CPU-D37
+FuelPump-Signal
 Text GLabel 1400 2700 0    50   Input ~ 0
-Fan-CPU-D27
+Fan-Signal
 Wire Wire Line
 	1400 2700 1550 2700
@@
 $EndComp
 Text GLabel 1650 1450 0    50   Input ~ 0
-TachoOut-CPU-D28
+TachoOut-Signal
 Text GLabel 2200 1650 2    50   Input ~ 0
 PowerGnd
@@
 	1    0    0    -1
 $EndComp
+Text GLabel 6350 1850 2    50   Input ~ 0
+BoostPWM-OUT
 Text GLabel 6350 1650 2    50   Input ~ 0
-BoostPWM-OUT
-Text GLabel 6350 1850 2    50   Input ~ 0
 IdlePWM-OUT
 Text GLabel 6350 1750 2    50   Input ~ 0
@@
 PowerGnd
 Text GLabel 4100 1650 0    50   Input ~ 0
-IdlePWM-CPU-D05
+IdlePWM-Signal
 Text GLabel 4100 1850 0    50   Input ~ 0
-BoostPWM-CPU-A21
+BoostPWM-Signal
 $Comp
 L Device:R R80
@@
 NoConn ~ 4650 1950
 Text GLabel 4350 2850 0    50   Input ~ 0
-Idle02
+Idle02-Signal
 NoConn ~ 4350 2850
 Text GLabel 4350 3150 0    50   Input ~ 0
-VVT
+VVT-Signal
 NoConn ~ 4350 3150
 Text GLabel 4900 2850 2    50   Input ~ 0

Commit message: MOSFET Drivers
Parts:
- removed IC11: VNLD5090-E, Package_SO:SO-8_5.3x6.2mm_P1.27mm, symbol VNLD5090-E:VNLD5090-E
- added IC11: VNS3NV04DP-E, SOIC127P600X175-8N, symbol Jag_Speedy-rescue:VNS3NV04DP-E-VNS3NV04DP-E
- Q1, Q2, Q3: symbol SSM3K357R:SSM3K357R,LF -> Jag_Speedy-rescue:SSM3K357R,LF-SSM3K357R
Connections:
- net BoostPWM-OUT: now also IC11.5 (DRAIN_2_1)
- net IdlePWM-OUT: now also IC11.7 (DRAIN_1_1)
- net PowerGnd: now also IC11.1 (SOURCE_1), IC11.3 (SOURCE_2); no longer R80.1, R81.2
- net at R82.2: now also IC11.2 (INPUT_1)
- net at R83.2: now also IC11.4 (INPUT_2)
- new net SignalGnd: R80.1, R81.2
Changed lines of the file:
@@
 $EndDescr
 $Comp
-L SSM3K357R:SSM3K357R,LF Q1
+L Jag_Speedy-rescue:SSM3K357R,LF-SSM3K357R Q1
 U 1 1 5F1A72FA
 P 1550 2700
@@
 $EndComp
 $Comp
-L SSM3K357R:SSM3K357R,LF Q2
+L Jag_Speedy-rescue:SSM3K357R,LF-SSM3K357R Q2
 U 1 1 5F1A78B8
 P 1600 4050
@@
 Fan
 $Comp
-L SSM3K357R:SSM3K357R,LF Q3
+L Jag_Speedy-rescue:SSM3K357R,LF-SSM3K357R Q3
 U 1 1 5F1AD432
 P 1650 1450
@@
 Text Notes 4250 950  0    118  ~ 0
 PWM Idle & Boost
-$Comp
-L VNLD5090-E:VNLD5090-E IC11
-U 1 1 5F1CC107
-P 4650 1650
-F 0 "IC11" H 5500 1915 50  0000 C CNN
-F 1 "VNLD5090-E" H 5500 1824 50  0000 C CNN
-F 2 "Package_SO:SO-8_5.3x6.2mm_P1.27mm" H 6200 1750 50  0001 L CNN
-F 3 "https://www.st.com/resource/en/datasheet/vnld5090-e.pdf" H 6200 1650 50  0001 L CNN
-F 4 "Gate Drivers OMNIFET III fully protect lo-side drvr" H 6200 1550 50  0001 L CNN "Description"
-F 5 "1.75" H 6200 1450 50  0001 L CNN "Height"
-F 6 "STMicroelectronics" H 6200 1350 50  0001 L CNN "Manufacturer_Name"
-F 7 "VNLD5090-E" H 6200 1250 50  0001 L CNN "Manufacturer_Part_Number"
-F 8 "VNLD5090-E" H 6200 1150 50  0001 L CNN "Arrow Part Number"
-F 9 "https://www.arrow.com/en/products/vnld5090-e/stmicroelectronics" H 6200 1050 50  0001 L CNN "Arrow Price/Stock"
-F 10 "511-VNLD5090-E" H 6200 950 50  0001 L CNN "Mouser Part Number"
-F 11 "https://www.mouser.com/Search/Refine.aspx?Keyword=511-VNLD5090-E" H 6200 850 50  0001 L CNN "Mouser Price/Stock"
-	1    4650 1650
-	1    0    0    -1
-$EndComp
-Text GLabel 6350 1850 2    50   Input ~ 0
-BoostPWM-OUT
-Text GLabel 6350 1650 2    50   Input ~ 0
-IdlePWM-OUT
-Text GLabel 6350 1750 2    50   Input ~ 0
-PowerGnd
-Text GLabel 6350 1950 2    50   Input ~ 0
-PowerGnd
-Text GLabel 4100 1650 0    50   Input ~ 0
-IdlePWM-Signal
-Text GLabel 4100 1850 0    50   Input ~ 0
-BoostPWM-Signal
-$Comp
-L Device:R R80
-U 1 1 5F1CCDB4
-P 4250 1500
-F 0 "R80" H 4320 1546 50  0000 L CNN
-F 1 "100k" H 4320 1455 50  0000 L CNN
-F 2 "Resistor_THT:R_Axial_DIN0207_L6.3mm_D2.5mm_P2.54mm_Vertical" V 4180 1500 50  0001 C CNN
-F 3 "~" H 4250 1500 50  0001 C CNN
-	1    4250 1500
-	1    0    0    -1
-$EndComp
-$Comp
-L Device:R R81
-U 1 1 5F1CD3E4
-P 4250 2000
-F 0 "R81" H 4320 2046 50  0000 L CNN
-F 1 "100k" H 4320 1955 50  0000 L CNN
-F 2 "Resistor_THT:R_Axial_DIN0207_L6.3mm_D2.5mm_P2.54mm_Vertical" V 4180 2000 50  0001 C CNN
-F 3 "~" H 4250 2000 50  0001 C CNN
-	1    4250 2000
-	1    0    0    -1
-$EndComp
-$Comp
-L Device:R R83
-U 1 1 5F1CD71C
-P 4500 1850
-F 0 "R83" V 4707 1850 50  0000 C CNN
-F 1 "1k" V 4616 1850 50  0000 C CNN
-F 2 "Resistor_THT:R_Axial_DIN0207_L6.3mm_D2.5mm_P2.54mm_Vertical" V 4430 1850 50  0001 C CNN
-F 3 "~" H 4500 1850 50  0001 C CNN
-	1    4500 1850
-	0    -1   -1   0
-$EndComp
-$Comp
-L Device:R R82
-U 1 1 5F1CDD62
-P 4500 1650
-F 0 "R82" V 4707 1650 50  0000 C CNN
-F 1 "1k" V 4616 1650 50  0000 C CNN
-F 2 "Resistor_THT:R_Axial_DIN0207_L6.3mm_D2.5mm_P2.54mm_Vertical" V 4430 1650 50  0001 C CNN
-F 3 "~" H 4500 1650 50  0001 C CNN
-	1    4500 1650
-	0    -1   -1   0
-$EndComp
-Text GLabel 4250 1200 2    50   Input ~ 0
-PowerGnd
-Text GLabel 4250 2300 2    50   Input ~ 0
-PowerGnd
-Wire Wire Line
-	4250 2300 4250 2150
-Wire Wire Line
-	4100 1850 4250 1850
-Wire Wire Line
-	4250 1650 4100 1650
-Wire Wire Line
-	4250 1350 4250 1200
-Wire Wire Line
-	4250 1650 4350 1650
-Connection ~ 4250 1650
-Wire Wire Line
-	4250 1850 4350 1850
-Connection ~ 4250 1850
-NoConn ~ 4650 1750
-NoConn ~ 4650 1950
 Text GLabel 4350 2850 0    50   Input ~ 0
 Idle02-Signal
@@
 NoConn ~ 4900 3150
 NoConn ~ 4900 2850
+$Comp
+L Jag_Speedy-rescue:VNS3NV04DP-E-VNS3NV04DP-E IC?
+U 1 1 5F04664C
+P 4650 1600
+AR Path="/5EF090BF/5F04664C" Ref="IC?"  Part="1"
+AR Path="/5F198969/5F04664C" Ref="IC11"  Part="1"
+F 0 "IC11" H 5450 1865 50  0000 C CNN
+F 1 "VNS3NV04DP-E" H 5450 1774 50  0000 C CNN
+F 2 "SOIC127P600X175-8N" H 6100 1700 50  0001 L CNN
+F 3 "https://www.st.com/resource/en/datasheet/vns3nv04dp-e.pdf" H 6100 1600 50  0001 L CNN
+F 4 "STMicroelectronics VNS3NV04DP-E Load Switch IC, 8-Pin, SOIC" H 6100 1500 50  0001 L CNN "Description"
+F 5 "1.75" H 6100 1400 50  0001 L CNN "Height"
+F 6 "STMicroelectronics" H 6100 1300 50  0001 L CNN "Manufacturer_Name"
+F 7 "VNS3NV04DP-E" H 6100 1200 50  0001 L CNN "Manufacturer_Part_Number"
+F 8 "VNS3NV04DP-E" H 6100 1100 50  0001 L CNN "Arrow Part Number"
+F 9 "https://www.arrow.com/en/products/vns3nv04dp-e/stmicroelectronics" H 6100 1000 50  0001 L CNN "Arrow Price/Stock"
+F 10 "511-VNS3NV04DP-E" H 6100 900 50  0001 L CNN "Mouser Part Number"
+F 11 "https://www.mouser.com/Search/Refine.aspx?Keyword=511-VNS3NV04DP-E" H 6100 800 50  0001 L CNN "Mouser Price/Stock"
+	1    4650 1600
+	1    0    0    -1
+$EndComp
+Text GLabel 4650 1800 0    50   Input ~ 0
+PowerGnd
+Text GLabel 4650 1600 1    50   Input ~ 0
+PowerGnd
+Text GLabel 6250 1900 2    50   Input ~ 0
+BoostPWM-OUT
+Text GLabel 6250 1700 2    50   Input ~ 0
+IdlePWM-OUT
+Text GLabel 4100 1900 0    50   Input ~ 0
+BoostPWM-Signal
+$Comp
+L Device:R R81
+U 1 1 5F0474F4
+P 4250 2050
+F 0 "R81" H 4050 2100 50  0000 L CNN
+F 1 "100k" H 4000 2000 50  0000 L CNN
+F 2 "Resistor_THT:R_Axial_DIN0207_L6.3mm_D2.5mm_P2.54mm_Vertical" V 4180 2050 50  0001 C CNN
+F 3 "~" H 4250 2050 50  0001 C CNN
+	1    4250 2050
+	1    0    0    -1
+$EndComp
+$Comp
+L Device:R R83
+U 1 1 5F0474FA
+P 4500 1900
+F 0 "R83" V 4300 1900 50  0000 C CNN
+F 1 "1k" V 4400 1900 50  0000 C CNN
+F 2 "Resistor_THT:R_Axial_DIN0207_L6.3mm_D2.5mm_P2.54mm_Vertical" V 4430 1900 50  0001 C CNN
+F 3 "~" H 4500 1900 50  0001 C CNN
+	1    4500 1900
+	0    -1   -1   0
+$EndComp
+Wire Wire Line
+	4100 1900 4250 1900
+Wire Wire Line
+	4250 1900 4350 1900
+Connection ~ 4250 1900
+Text GLabel 4250 2200 0    50   Input ~ 0
+SignalGnd
+Connection ~ 4250 1700
+Wire Wire Line
+	4250 1700 4350 1700
+Wire Wire Line
+	4250 1700 4100 1700
+$Comp
+L Device:R R82
+U 1 1 5F049205
+P 4500 1700
+F 0 "R82" V 4707 1700 50  0000 C CNN
+F 1 "1k" V 4616 1700 50  0000 C CNN
+F 2 "Resistor_THT:R_Axial_DIN0207_L6.3mm_D2.5mm_P2.54mm_Vertical" V 4430 1700 50  0001 C CNN
+F 3 "~" H 4500 1700 50  0001 C CNN
+	1    4500 1700
+	0    -1   -1   0
+$EndComp
+$Comp
+L Device:R R80
+U 1 1 5F0491FF
+P 4250 1550
+F 0 "R80" H 4050 1600 50  0000 L CNN
+F 1 "100k" H 4000 1500 50  0000 L CNN
+F 2 "Resistor_THT:R_Axial_DIN0207_L6.3mm_D2.5mm_P2.54mm_Vertical" V 4180 1550 50  0001 C CNN
+F 3 "~" H 4250 1550 50  0001 C CNN
+	1    4250 1550
+	1    0    0    -1
+$EndComp
+Text GLabel 4100 1700 0    50   Input ~ 0
+IdlePWM-Signal
+NoConn ~ 6250 1800
+NoConn ~ 6250 1600
+Text GLabel 4250 1400 0    50   Input ~ 0
+SignalGnd
 $EndSCHEMATC

Commit message: Rationalise level shifting
Parts:
- IC11: footprint SOIC127P600X175-8N -> Package_SO:SO-8_3.9x4.9mm_P1.27mm; symbol Jag_Speedy-rescue:VNS3NV04DP-E-VNS3NV04DP-E -> Jag_Speedy-rescue:VNS3NV04DP-E-VNS3NV04DP-E-Jag_Speedy-rescue
- Q1, Q2, Q3: symbol Jag_Speedy-rescue:SSM3K357R,LF-SSM3K357R -> Jag_Speedy-rescue:SSM3K357R,LF-SSM3K357R-Jag_Speedy-rescue
Connections:
- net BoostPWM-OUT: no longer IC11.5 (DRAIN_2_1)
- net BoostPWM-Signal: no longer R81.1, R83.1
- new net CCPump-OUT: IC11.5 (DRAIN_2_1)
- new net CCPump-Signal: R81.1, R83.1
Changed lines of the file:
@@
 $EndDescr
 $Comp
-L Jag_Speedy-rescue:SSM3K357R,LF-SSM3K357R Q1
+L Jag_Speedy-rescue:SSM3K357R,LF-SSM3K357R-Jag_Speedy-rescue Q1
 U 1 1 5F1A72FA
 P 1550 2700
@@
 $EndComp
 $Comp
-L Jag_Speedy-rescue:SSM3K357R,LF-SSM3K357R Q2
+L Jag_Speedy-rescue:SSM3K357R,LF-SSM3K357R-Jag_Speedy-rescue Q2
 U 1 1 5F1A78B8
 P 1600 4050
@@
 Fan
 $Comp
-L Jag_Speedy-rescue:SSM3K357R,LF-SSM3K357R Q3
+L Jag_Speedy-rescue:SSM3K357R,LF-SSM3K357R-Jag_Speedy-rescue Q3
 U 1 1 5F1AD432
 P 1650 1450
@@
 Idle02-Signal
 NoConn ~ 4350 2850
-Text GLabel 4350 3150 0    50   Input ~ 0
-VVT-Signal
+Text GLabel 4100 1900 0    50   Input ~ 0
+CCPump-Signal
 NoConn ~ 4350 3150
 Text GLabel 4900 2850 2    50   Input ~ 0
 Idle02-OUT
-Text GLabel 4900 3150 2    50   Input ~ 0
-VVT-OUT
+Text GLabel 6250 1900 2    50   Input ~ 0
+CCPump-OUT
 NoConn ~ 4900 3150
 NoConn ~ 4900 2850
 $Comp
-L Jag_Speedy-rescue:VNS3NV04DP-E-VNS3NV04DP-E IC?
+L Jag_Speedy-rescue:VNS3NV04DP-E-VNS3NV04DP-E-Jag_Speedy-rescue IC?
 U 1 1 5F04664C
 P 4650 1600
@@
 F 0 "IC11" H 5450 1865 50  0000 C CNN
 F 1 "VNS3NV04DP-E" H 5450 1774 50  0000 C CNN
-F 2 "SOIC127P600X175-8N" H 6100 1700 50  0001 L CNN
+F 2 "Package_SO:SO-8_3.9x4.9mm_P1.27mm" H 6100 1700 50  0001 L CNN
 F 3 "https://www.st.com/resource/en/datasheet/vns3nv04dp-e.pdf" H 6100 1600 50  0001 L CNN
 F 4 "STMicroelectronics VNS3NV04DP-E Load Switch IC, 8-Pin, SOIC" H 6100 1500 50  0001 L CNN "Description"
@@
 Text GLabel 4650 1600 1    50   Input ~ 0
 PowerGnd
-Text GLabel 6250 1900 2    50   Input ~ 0
+Text GLabel 4900 3150 2    50   Input ~ 0
 BoostPWM-OUT
 Text GLabel 6250 1700 2    50   Input ~ 0
 IdlePWM-OUT
-Text GLabel 4100 1900 0    50   Input ~ 0
+Text GLabel 4350 3150 0    50   Input ~ 0
 BoostPWM-Signal
 $Comp

Commit message: SMD Update
Parts:
- Q1, Q2, Q3: footprint Package_TO_SOT_THT:TO-3P-3_Vertical -> Package_TO_SOT_SMD:SOT-23
- R80, R81, R82, R83: footprint Resistor_THT:R_Axial_DIN0207_L6.3mm_D2.5mm_P2.54mm_Vertical -> Resistor_SMD:R_0805_2012Metric
Other:
- note added: "PWM Idle & Charge Cooler Pump"
- note removed: "PWM Idle & Boost"
Changed lines of the file:
@@
 F 0 "Q1" H 1980 2846 50  0000 L CNN
 F 1 "SSM3K357R,LF" H 1980 2755 50  0000 L CNN
-F 2 "Package_TO_SOT_THT:TO-3P-3_Vertical" H 2000 2650 50  0001 L CNN
+F 2 "Package_TO_SOT_SMD:SOT-23" H 2000 2650 50  0001 L CNN
 F 3 "https://toshiba.semicon-storage.com/info/docget.jsp?did=59207&prodName=SSM3K357R" H 2000 2550 50  0001 L CNN
 F 4 "MOSFET LowON Res MOSFET ID=.65A VDSS=60V" H 2000 2450 50  0001 L CNN "Description"
@@
 F 0 "Q2" H 2030 4196 50  0000 L CNN
 F 1 "SSM3K357R,LF" H 2030 4105 50  0000 L CNN
-F 2 "Package_TO_SOT_THT:TO-3P-3_Vertical" H 2050 4000 50  0001 L CNN
+F 2 "Package_TO_SOT_SMD:SOT-23" H 2050 4000 50  0001 L CNN
 F 3 "https://toshiba.semicon-storage.com/info/docget.jsp?did=59207&prodName=SSM3K357R" H 2050 3900 50  0001 L CNN
 F 4 "MOSFET LowON Res MOSFET ID=.65A VDSS=60V" H 2050 3800 50  0001 L CNN "Description"
@@
 F 0 "Q3" H 2080 1596 50  0000 L CNN
 F 1 "SSM3K357R,LF" H 2080 1505 50  0000 L CNN
-F 2 "Package_TO_SOT_THT:TO-3P-3_Vertical" H 2100 1400 50  0001 L CNN
+F 2 "Package_TO_SOT_SMD:SOT-23" H 2100 1400 50  0001 L CNN
 F 3 "https://toshiba.semicon-storage.com/info/docget.jsp?did=59207&prodName=SSM3K357R" H 2100 1300 50  0001 L CNN
 F 4 "MOSFET LowON Res MOSFET ID=.65A VDSS=60V" H 2100 1200 50  0001 L CNN "Description"
@@
 Fuel Pump
 Text Notes 4250 950  0    118  ~ 0
-PWM Idle & Boost
+PWM Idle & Charge Cooler Pump
 Text GLabel 4350 2850 0    50   Input ~ 0
 Idle02-Signal
@@
 F 0 "R81" H 4050 2100 50  0000 L CNN
 F 1 "100k" H 4000 2000 50  0000 L CNN
-F 2 "Resistor_THT:R_Axial_DIN0207_L6.3mm_D2.5mm_P2.54mm_Vertical" V 4180 2050 50  0001 C CNN
+F 2 "Resistor_SMD:R_0805_2012Metric" V 4180 2050 50  0001 C CNN
 F 3 "~" H 4250 2050 50  0001 C CNN
 	1    4250 2050
@@
 F 0 "R83" V 4300 1900 50  0000 C CNN
 F 1 "1k" V 4400 1900 50  0000 C CNN
-F 2 "Resistor_THT:R_Axial_DIN0207_L6.3mm_D2.5mm_P2.54mm_Vertical" V 4430 1900 50  0001 C CNN
+F 2 "Resistor_SMD:R_0805_2012Metric" V 4430 1900 50  0001 C CNN
 F 3 "~" H 4500 1900 50  0001 C CNN
 	1    4500 1900
@@
 F 0 "R82" V 4707 1700 50  0000 C CNN
 F 1 "1k" V 4616 1700 50  0000 C CNN
-F 2 "Resistor_THT:R_Axial_DIN0207_L6.3mm_D2.5mm_P2.54mm_Vertical" V 4430 1700 50  0001 C CNN
+F 2 "Resistor_SMD:R_0805_2012Metric" V 4430 1700 50  0001 C CNN
 F 3 "~" H 4500 1700 50  0001 C CNN
 	1    4500 1700
@@
 F 0 "R80" H 4050 1600 50  0000 L CNN
 F 1 "100k" H 4000 1500 50  0000 L CNN
-F 2 "Resistor_THT:R_Axial_DIN0207_L6.3mm_D2.5mm_P2.54mm_Vertical" V 4180 1550 50  0001 C CNN
+F 2 "Resistor_SMD:R_0805_2012Metric" V 4180 1550 50  0001 C CNN
 F 3 "~" H 4250 1550 50  0001 C CNN
 	1    4250 1550
