File: reference/hardware/v0.3/Jag_Speedy/power.sch (KiCad schematic (older format))
At the start: 8 parts, among them IC9 LM2940T-5.0_NOPB

Commit message: Schematic pin mapping
Changed lines of the file:
@@
 	1    0    0    -1
 $EndComp
-Text GLabel 6300 2950 2    50   Output ~ 0
+Text GLabel 5900 2800 1    50   Output ~ 0
 5V
 Text GLabel 2800 2950 0    50   Input ~ 0
@@
 Text GLabel 3200 2750 1    50   Output ~ 0
 12V
-Wire Wire Line
-	4750 2950 4750 3850
 Wire Wire Line
 	4750 3850 4300 3850
@@
 	5450 2950 5900 2950
 Connection ~ 5450 2950
-Wire Wire Line
-	5900 2950 6300 2950
-Connection ~ 5900 2950
-Text GLabel 4750 3950 3    50   Output ~ 0
+Text GLabel 4750 3950 3    50   Input ~ 0
 PowerGnd
 Wire Wire Line
@@
 Wire Wire Line
 	3900 3850 3050 3850
+Connection ~ 5900 2950
+Wire Wire Line
+	5900 2800 5900 2950
+Wire Wire Line
+	4750 2950 4750 3850
 $EndSCHEMATC

Commit message: MOSFET Drivers
Parts:
- D20: symbol 1N5919BG:1N5919BG -> Jag_Speedy-rescue:1N5919BG-1N5919BG
- IC9: symbol LM2940T:LM2940T-5.0_NOPB -> Jag_Speedy-rescue:LM2940T-5.0_NOPB-LM2940T
- RV1: symbol ERZV14D220:ERZV14D220 -> Jag_Speedy-rescue:ERZV14D220-ERZV14D220
Changed lines of the file:
@@
 $EndDescr
 $Comp
-L LM2940T:LM2940T-5.0_NOPB IC9
+L Jag_Speedy-rescue:LM2940T-5.0_NOPB-LM2940T IC9
 U 1 1 5EFCE38E
 P 4650 2950
@@
 $EndComp
 $Comp
-L ERZV14D220:ERZV14D220 RV1
+L Jag_Speedy-rescue:ERZV14D220-ERZV14D220 RV1
 U 1 1 5EFCEC0A
 P 3050 2950
@@
 $EndComp
 $Comp
-L 1N5919BG:1N5919BG D20
+L Jag_Speedy-rescue:1N5919BG-1N5919BG D20
 U 1 1 5EFD0FB3
 P 5900 2950
+AR Path="/5EFD0FB3" Ref="D20"  Part="1"
+AR Path="/5EF0923F/5EFD0FB3" Ref="D20"  Part="1"
 F 0 "D20" V 6154 3078 50  0000 L CNN
 F 1 "1N5919BG" V 6245 3078 50  0000 L CNN

Commit message: Rationalise level shifting
Parts:
- D20: symbol Jag_Speedy-rescue:1N5919BG-1N5919BG -> Jag_Speedy-rescue:1N5919BG-1N5919BG-Jag_Speedy-rescue
- IC9: symbol Jag_Speedy-rescue:LM2940T-5.0_NOPB-LM2940T -> Jag_Speedy-rescue:LM2940T-5.0_NOPB-LM2940T-Jag_Speedy-rescue
- RV1: symbol Jag_Speedy-rescue:ERZV14D220-ERZV14D220 -> Jag_Speedy-rescue:ERZV14D220-ERZV14D220-Jag_Speedy-rescue
Changed lines of the file:
@@
 $EndDescr
 $Comp
-L Jag_Speedy-rescue:LM2940T-5.0_NOPB-LM2940T IC9
+L Jag_Speedy-rescue:LM2940T-5.0_NOPB-LM2940T-Jag_Speedy-rescue IC9
 U 1 1 5EFCE38E
 P 4650 2950
@@
 $EndComp
 $Comp
-L Jag_Speedy-rescue:ERZV14D220-ERZV14D220 RV1
+L Jag_Speedy-rescue:ERZV14D220-ERZV14D220-Jag_Speedy-rescue RV1
 U 1 1 5EFCEC0A
 P 3050 2950
@@
 $EndComp
 $Comp
-L Jag_Speedy-rescue:1N5919BG-1N5919BG D20
+L Jag_Speedy-rescue:1N5919BG-1N5919BG-Jag_Speedy-rescue D20
 U 1 1 5EFD0FB3
 P 5900 2950

Commit message: SMD Update
Parts:
- added C33: 4.7nF, Capacitor_SMD:C_0805_2012Metric, symbol Device:C
- added D21: 1N5818, Diode_SMD:D_SMA, symbol Diode:1N5818
- added R9: 10K, Resistor_SMD:R_0805_2012Metric, symbol Device:R
- C29: footprint Capacitor_THT:CP_Radial_D5.0mm_P2.50mm -> Capacitor_Tantalum_SMD:CP_EIA-7343-31_Kemet-D
- C30, C31: footprint Capacitor_THT:CP_Radial_D5.0mm_P2.50mm -> Capacitor_SMD:C_0805_2012Metric
- C32: footprint Capacitor_THT:CP_Radial_D5.0mm_P2.50mm -> Capacitor_Tantalum_SMD:CP_EIA-3528-21_Kemet-B
- D19: footprint Diode_THT:D_DO-41_SOD81_P10.16mm_Horizontal -> Diode_SMD:D_SMA
- D20: footprint Diode_THT:D_DO-35_SOD27_P10.16mm_Horizontal -> Diode_SMD:D_SMB
- IC9: footprint Package_TO_SOT_THT:TO-3P-3_Vertical -> Package_TO_SOT_SMD:TO-263-3_TabPin2
- RV1: footprint Varistor:RV_Disc_D7mm_W5.7mm_P5mm -> Varistor:RV_Disc_D15.5mm_W4.7mm_P7.5mm
Connections:
- net 5V: now also D21.1 (K), R9.1
- net PowerGnd: now also C33.2
- new net Reset: C33.1, D21.2 (A), R9.2
Other:
- note added: "Reset\nProtection"
- moved on the sheet: C29, C30, C31, C32, D20, RV1
