File: reference/hardware/v0.3/Jag_Speedy/Jag_Speedy.kicad_pcb (KiCad board)
At the start: 2 copper layers, 215 parts, among them IC1 MPX4250AP, IC10 SP720APP, IC11 VNLD5090-E, IC11 VNS3NV04DP-E, IC2 MPX4250AP, IC3 VNLD5090-E, IC3 VNS3NV04DP-E, IC4 VNLD5090-E, IC4 VNS3NV04DP-E, IC5 VNLD5090-E, IC5 VNS3NV04DP-E, IC6 TC4424EPA, IC7 TC4424EPA, IC8 TC4424EPA, IC9 LM2940T-5.0_NOPB, J1 Inputs, J2 Ouputs01, J3 Outputs02, J4 Power, J5 Bluetooth, J6 Dual VR Conditioner, J7 Canbus, Q1 SSM3K357R,LF, Q2 SSM3K357R,LF, Q3 SSM3K357R,LF, U1 LMV324, U2 LMV324, U3 Teensy 3.5, U4 LMV324, U5 SN65HVD230

Commit message: PCB Update
Parts:
- removed De: 1N4004, Diode_THT:D_DO-41_SOD81_P10.16mm_Horizontal
- removed R10, R11, R12, R86, R87, R88, R89, R9: 330k, Resistor_THT:R_Axial_DIN0207_L6.3mm_D2.5mm_P2.54mm_Vertical
- removed R13, R14, R15, R16, R84, R85, R90, R91: 180k, Resistor_THT:R_Axial_DIN0207_L6.3mm_D2.5mm_P2.54mm_Vertical
- removed U2, U4: LMV324, Package_DIP:DIP-14_W7.62mm_Socket
- added IC12: SP720APP, Package_DIP:DIP-16_W7.62mm, F.Cu at (151.0, 114.6)
- added R1: 180k, Resistor_THT:R_Axial_DIN0207_L6.3mm_D2.5mm_P2.54mm_Vertical, F.Cu at (174.0, 114.6)
- added R2: 180k, Resistor_THT:R_Axial_DIN0207_L6.3mm_D2.5mm_P2.54mm_Vertical, F.Cu at (180.1, 114.6)
- added R3: 330k, Resistor_THT:R_Axial_DIN0207_L6.3mm_D2.5mm_P2.54mm_Vertical, F.Cu at (174.0, 118.6)
- added R4: 330k, Resistor_THT:R_Axial_DIN0207_L6.3mm_D2.5mm_P2.54mm_Vertical, F.Cu at (180.1, 118.6)
- added R5: 330k, Resistor_THT:R_Axial_DIN0207_L6.3mm_D2.5mm_P2.54mm_Vertical, F.Cu at (174.0, 122.7)
- added R6: 330k, Resistor_THT:R_Axial_DIN0207_L6.3mm_D2.5mm_P2.54mm_Vertical, F.Cu at (186.3, 114.6)
- added R7: 180k, Resistor_THT:R_Axial_DIN0207_L6.3mm_D2.5mm_P2.54mm_Vertical, F.Cu at (174.0, 126.7)
- added R8: 180k, Resistor_THT:R_Axial_DIN0207_L6.3mm_D2.5mm_P2.54mm_Vertical, F.Cu at (180.1, 122.7)
- added U1: LMV324, Package_DIP:DIP-14_W7.62mm_Socket, F.Cu at (162.3, 114.7)
- IC11, IC3, IC4, IC5: value VNLD5090-E -> VNS3NV04DP-E; footprint Package_SO:SO-8_5.3x6.2mm_P1.27mm -> Package_SO:SO-8_3.9x4.9mm_P1.27mm
- J2: footprint Connector_PinHeader_1.00mm:PinHeader_2x06_P1.00mm_Horizontal -> Connector_PinHeader_1.00mm:PinHeader_2x07_P1.00mm_Horizontal
- R3, R4: value 180k -> 330k
- R7, R8: value 330k -> 180k
- moved J2 42.3 mm to (-40.6, 62.2)
- moved R39 32.4 mm to (-2.54, 29.2)
- moved R44 26.2 mm to (6.35, 35.6), turned to 180 degrees
- moved R38 25.4 mm to (3.81, 29.2), turned to 0 degrees
- moved R45 24.4 mm to (-2.54, 35.6), turned to 0 degrees
- moved IC5 11.4 mm to (0.00, 76.2)
- moved D9 10.2 mm to (-11.4, 57.1), turned to 180 degrees
- moved IC4 6.35 mm to (0.00, 61.0)
- moved IC3 1.27 mm to (0.00, 45.7)
Connections:
- IC1 pad 4: Net-(IC1-Pad4) -> (no net)
- IC1 pad 5: Net-(IC1-Pad5) -> (no net)
- IC1 pad 6: Net-(IC1-Pad6) -> (no net)
- IC10 pad 10: ADCClamp09 -> (no net)
- IC10 pad 11: ADCClamp10 -> (no net)
- IC10 pad 12: ADCClamp11 -> (no net)
- IC10 pad 13: Net-(IC10-Pad13) -> (no net)
- IC10 pad 14: Net-(IC10-Pad14) -> (no net)
- IC10 pad 15: Net-(IC10-Pad15) -> (no net)
- IC10 pad 5: ADCClamp05 -> (no net)
- IC11 pad 1: Net-(IC11-Pad1) -> PowerGnd
- IC11 pad 3: Net-(IC11-Pad3) -> PowerGnd
- IC11 pad 5: PowerGnd -> CCPump-OUT
- IC11 pad 6: IdlePWM-OUT -> Net-(IC11-Pad6)
- IC11 pad 7: PowerGnd -> IdlePWM-OUT
- IC11 pad 8: BoostPWM-OUT -> Net-(IC11-Pad8)
- IC2 pad 4: Net-(IC2-Pad4) -> (no net)
- IC2 pad 5: Net-(IC2-Pad5) -> (no net)
- IC2 pad 6: Net-(IC2-Pad6) -> (no net)
- IC3 pad 1: Net-(IC3-Pad1) -> PowerGnd
- IC3 pad 3: Net-(IC3-Pad3) -> PowerGnd
- IC3 pad 5: PowerGnd -> Inj02-OUT
- IC3 pad 6: Inj02-OUT -> Net-(IC3-Pad6)
- IC3 pad 7: PowerGnd -> Inj01-OUT
- IC3 pad 8: Inj01-OUT -> Net-(IC3-Pad8)
- IC4 pad 1: Net-(IC4-Pad1) -> PowerGnd
- IC4 pad 3: Net-(IC4-Pad3) -> PowerGnd
- IC4 pad 5: PowerGnd -> Inj04-OUT
- IC4 pad 6: Inj04-OUT -> Net-(IC4-Pad6)
- IC4 pad 7: PowerGnd -> Inj03-OUT
- IC4 pad 8: Inj03-OUT -> Net-(IC4-Pad8)
- IC5 pad 1: Net-(IC5-Pad1) -> PowerGnd
- IC5 pad 3: Net-(IC5-Pad3) -> PowerGnd
- IC5 pad 5: PowerGnd -> Inj06-OUT
- IC5 pad 6: Inj06-OUT -> Net-(IC5-Pad6)
- IC5 pad 7: PowerGnd -> Inj05-OUT
- IC5 pad 8: Inj05-OUT -> Net-(IC5-Pad8)
- IC6 pad 1: Net-(IC6-Pad1) -> (no net)
- IC6 pad 8: Net-(IC6-Pad8) -> (no net)
- IC7 pad 1: Net-(IC7-Pad1) -> (no net)
- IC7 pad 8: Net-(IC7-Pad8) -> (no net)
- IC8 pad 1: Net-(IC8-Pad1) -> (no net)
- IC8 pad 8: Net-(IC8-Pad8) -> (no net)
- J1 pad 1: Net-(J1-Pad1) -> 3V3
- J1 pad 12: 5V -> 3V3
- J2 pad 1: Inj01-OUT -> PowerGnd
- J2 pad 10: Ign04-OUT -> Ign03-OUT
- J2 pad 11: Ign05-OUT -> Ign04-OUT
- J2 pad 12: Ign06-OUT -> Ign05-OUT
- J2 pad 2: Inj02-OUT -> Inj01-OUT
- J2 pad 3: Inj03-OUT -> Inj02-OUT
- J2 pad 4: Inj04-OUT -> Inj03-OUT
- J2 pad 5: Inj05-OUT -> Inj04-OUT
- J2 pad 6: Inj06-OUT -> Inj05-OUT
- J2 pad 7: Ign01-OUT -> Inj06-OUT
- J2 pad 8: Ign02-OUT -> Ign01-OUT
- J2 pad 9: Ign03-OUT -> Ign02-OUT
- J3 pad 1: BoostPWM-OUT -> (no net)
- J3 pad 10: Net-(J3-Pad10) -> PowerGnd
- J3 pad 3: Net-(J3-Pad3) -> PowerGnd
- J3 pad 7: Idle02-OUT -> (no net)
- J3 pad 9: Net-(J3-Pad9) -> PowerGnd
- J5 pad 5: Net-(J5-Pad5) -> (no net)
- J5 pad 6: Net-(J5-Pad6) -> (no net)
- R1 pad 1: ADCClamp09 -> ADCClamp06
- R2 pad 1: ADCClamp06 -> ADCClamp07
- R23 pad 1: 5V -> 3V3
- R24 pad 1: 5V -> 3V3
- R25 pad 1: 5V -> 3V3
- R26 pad 1: 5V -> 3V3
- R3 pad 1: ADCClamp07 -> Net-(R2-Pad2)
- R3 pad 2: Net-(R3-Pad2) -> PowerGnd
- R38 pad 2: Inj01-CPU-D08 -> CPU-D08
- R39 pad 1: Inj02-CPU-D09 -> CPU-D09
- R4 pad 1: ADCClamp11 -> Net-(R1-Pad2)
- R4 pad 2: Net-(R4-Pad2) -> PowerGnd
- R40 pad 1: PowerGnd -> CPU-D10
- R40 pad 2: Inj03-CPU-D10 -> PowerGnd
- R41 pad 1: Inj04-CPU-D11 -> CPU-D11
- R42 pad 2: Inj05-CPU-D12 -> CPU-D12
- R43 pad 1: Inj06-CPU-D07 -> CPU-D13
- R44 pad 1: Inj01-CPU-D08 -> CPU-D08
- R44 pad 2: Net-(IC3-Pad1) -> Net-(IC3-Pad2)
- R45 pad 1: Inj02-CPU-D09 -> CPU-D09
- R45 pad 2: Net-(IC3-Pad3) -> Net-(IC3-Pad4)
- R46 pad 1: Inj03-CPU-D10 -> CPU-D10
- R46 pad 2: Net-(IC4-Pad1) -> Net-(IC4-Pad2)
- R47 pad 1: Inj04-CPU-D11 -> CPU-D11
- R47 pad 2: Net-(IC4-Pad3) -> Net-(IC4-Pad4)
- R48 pad 1: Inj05-CPU-D12 -> CPU-D12
- R48 pad 2: Net-(IC5-Pad1) -> Net-(IC5-Pad2)
- R49 pad 1: Inj06-CPU-D07 -> CPU-D13
- R49 pad 2: Net-(IC5-Pad3) -> Net-(IC5-Pad4)
- R5 pad 1: Net-(R1-Pad2) -> PowerGnd
- R5 pad 2: PowerGnd -> Net-(R5-Pad2)
- R6 pad 1: Net-(R2-Pad2) -> PowerGnd
- R6 pad 2: PowerGnd -> Net-(R6-Pad2)
- R7 pad 1: Net-(R3-Pad2) -> Net-(R5-Pad2)
- R7 pad 2: PowerGnd -> ADCClamp03
- R8 pad 1: Net-(R4-Pad2) -> Net-(R6-Pad2)
- R8 pad 2: PowerGnd -> ADCClamp04
- R80 pad 2: IdlePWM-CPU-D05 -> CPU-D05
- R81 pad 1: BoostPWM-CPU-A21 -> CCPump-Signal
- R82 pad 1: IdlePWM-CPU-D05 -> CPU-D05
- R82 pad 2: Net-(IC11-Pad1) -> Net-(IC11-Pad2)
- R83 pad 1: BoostPWM-CPU-A21 -> CCPump-Signal
- R83 pad 2: Net-(IC11-Pad3) -> Net-(IC11-Pad4)
- U1 pad 1: CPU-A0 -> CPU-A8
- U1 pad 10: Net-(R10-Pad2) -> Net-(R6-Pad2)
- U1 pad 12: Net-(R2-Pad2) -> Net-(R1-Pad2)
- U1 pad 2: CPU-A0 -> CPU-A8
- U1 pad 3: Net-(R13-Pad1) -> Net-(R5-Pad2)
- U1 pad 5: Net-(R1-Pad2) -> Net-(R2-Pad2)
- U1 pad 6: CLT-Signal-3.3V -> Barro-Signal-3.3V
- U1 pad 7: CLT-Signal-3.3V -> Barro-Signal-3.3V
- U3 pad 18: Net-(U3-Pad18) -> (no net)
- U3 pad 22: Net-(U3-Pad22) -> (no net)
- U3 pad 25: Net-(U3-Pad25) -> (no net)
- U3 pad 28: Net-(U3-Pad28) -> (no net)
- U3 pad 29: Net-(U3-Pad29) -> (no net)
- U3 pad 30: Net-(U3-Pad30) -> (no net)
- U3 pad 31: Net-(U3-Pad31) -> (no net)
- U3 pad 37: Net-(U3-Pad37) -> (no net)
- U3 pad 38: Net-(U3-Pad38) -> (no net)
- U3 pad 4: Net-(U3-Pad4) -> (no net)
- U3 pad 41: CPU-A0 -> ADCClamp08
- U3 pad 42: CLT-Signal-3.3V -> ADCClamp09
- U3 pad 45: BRV-Signal-3.3V -> ADCClamp05
- U3 pad 47: Net-(U3-Pad47) -> (no net)
- U3 pad 51: Net-(U3-Pad51) -> (no net)
- U3 pad 54: Net-(U3-Pad54) -> (no net)
- U3 pad 55: Net-(U3-Pad55) -> (no net)
- U3 pad 56: CPU-A10 -> ADCClamp10
- U3 pad 57: CPU-A11 -> ADCClamp11
- U3 pad 58: Net-(U3-Pad58) -> (no net)
- U3 pad 59: Net-(U3-Pad59) -> (no net)
- U3 pad 62: Net-(U3-Pad62) -> (no net)
- U3 pad 8: CPU-D06 -> (no net)
- U3 pad 9: BoostPWM-Signal -> (no net)
- U5 pad 5: Net-(U5-Pad5) -> (no net)

Commit message: SMD Update
Parts:
- removed the D1 at (121.9, 36.8)
- removed the D1 at (-25.4, 41.9)
- removed the D10 at (99.4, 16.1)
- removed the D10 at (-11.4, 64.8)
- removed the D11 at (85.5, 20.3)
- removed the D11 at (-11.4, 72.4)
- removed the D12 at (85.5, 16.1)
- removed the D12 at (-11.4, 80.0)
- removed the D2 at (126.3, 30.4)
- removed the D2 at (-25.4, 49.5)
- removed the D3 at (116.0, 36.8)
- removed the D3 at (-25.4, 57.1)
- removed the D4 at (120.4, 31.3)
- removed the D4 at (-25.4, 64.8)
- removed the D5 at (125.4, 24.8)
- removed the D5 at (-25.4, 72.4)
- removed the D6 at (114.5, 31.3)
- removed the D6 at (-25.4, 80.0)
- removed the D8 at (99.4, 20.3)
- removed the D8 at (-11.4, 49.5)
- removed the D9 at (85.5, 24.6)
- removed the D9 at (-11.4, 57.1)
- removed the IC11 at (195.6, 146.1)
- removed the IC11 at (140.9, 17.2)
- removed the IC3 at (0.00, 45.7)
- removed the IC3 at (96.3, 34.2)
- removed the IC4 at (0.00, 61.0)
- removed the IC4 at (115.7, 17.2)
- removed the IC5 at (0.00, 76.2)
- removed the IC5 at (87.9, 34.2)
- removed the R1 at (174.0, 114.6)
- removed the R1 at (121.1, 131.1)
- removed the R2 at (180.1, 114.6)
- removed the R2 at (154.5, 89.2)
- removed the R3 at (174.0, 118.6)
- removed the R3 at (160.6, 89.2)
- removed the R38 at (99.6, 24.5)
- removed the R38 at (3.81, 29.2)
- removed the R39 at (105.7, 24.5)
- removed the R39 at (-2.54, 29.2)
- removed the R4 at (180.1, 118.6)
- removed the R4 at (154.5, 93.2)
- removed the R40 at (91.8, 39.4)
- removed the R40 at (24.6, 72.4)
- removed the R41 at (85.7, 39.4)
- removed the R41 at (8.89, 72.4)
- removed the R42 at (113.5, 22.4)
- removed the R42 at (47.0, 48.3)
- removed the R43 at (105.7, 28.5)
- removed the R43 at (44.5, 54.6)
- removed the R44 at (110.2, 36.6)
- removed the R44 at (6.35, 35.6)
- removed the R45 at (104.1, 36.6)
- removed the R45 at (-2.54, 35.6)
- removed the R46 at (99.6, 28.5)
- removed the R46 at (26.7, 64.8)
- removed the R47 at (125.8, 20.0)
- removed the R47 at (8.89, 64.8)
- removed the R48 at (118.0, 26.5)
- removed the R48 at (49.5, 63.5)
- removed the R49 at (128.1, 16.0)
- removed the R49 at (38.1, 54.6)
- removed the R5 at (174.0, 122.7)
- removed the R5 at (138.4, 105.4)
- removed the R50 at (108.7, 32.6)
- removed the R50 at (-34.3, 41.9)
- removed the R51 at (119.6, 22.4)
- removed the R51 at (-34.3, 49.5)
- removed the R52 at (111.9, 26.5)
- removed the R52 at (-34.3, 57.1)
- removed the R53 at (98.0, 39.4)
- removed the R53 at (-34.3, 64.8)
- removed the R54 at (121.9, 16.0)
- removed the R54 at (-34.3, 72.4)
- removed the R55 at (102.6, 32.6)
- removed the R55 at (-34.3, 80.0)
- removed the R6 at (186.3, 114.6)
- removed the R6 at (160.6, 93.2)
- removed the R7 at (174.0, 126.7)
- removed the R7 at (154.5, 97.3)
- removed the R8 at (180.1, 122.7)
- removed the R8 at (138.4, 100.3)
- removed the R80 at (150.9, 20.0)
- removed the R80 at (223.0, 119.0)
- removed the R81 at (138.7, 22.4)
- removed the R81 at (216.8, 119.0)
- removed the R82 at (147.1, 16.0)
- removed the R82 at (199.4, 138.4)
- removed the R83 at (144.8, 22.4)
- removed the R83 at (193.0, 138.4)
- removed the U1 at (162.3, 114.7)
- removed the U1 at (205.7, 121.9)
- added C33: 4.7nF, Capacitor_SMD:C_0805_2012Metric, F.Cu at (141.8, -5.37)
- added D1: LED, LED_SMD:LED_0805_2012Metric, F.Cu at (83.5, 53.3)
- added D10: 1N4004, Diode_SMD:D_SOD-323, F.Cu at (76.2, 58.4)
- added D11: 1N4004, Diode_SMD:D_SOD-323, F.Cu at (76.2, 71.1)
- added D12: 1N4004, Diode_SMD:D_SOD-323, F.Cu at (76.2, 67.3)
- added D2: LED, LED_SMD:LED_0805_2012Metric, F.Cu at (83.5, 49.5)
- added D21: 1N5818, Diode_SMD:D_SMA, F.Cu at (135.6, -4.57)
- added D3: LED, LED_SMD:LED_0805_2012Metric, F.Cu at (83.8, 62.2)
- added D4: LED, LED_SMD:LED_0805_2012Metric, F.Cu at (83.5, 58.4)
- added D5: LED, LED_SMD:LED_0805_2012Metric, F.Cu at (83.5, 72.4)
- added D6: LED, LED_SMD:LED_0805_2012Metric, F.Cu at (83.5, 67.3)
- added D8: 1N4004, Diode_SMD:D_SOD-323, F.Cu at (76.2, 49.5)
- added D9: 1N4004, Diode_SMD:D_SOD-323, F.Cu at (76.2, 62.2)
- added IC11: VNS3NV04DP-E, Package_SO:SO-8_3.9x4.9mm_P1.27mm, F.Cu at (228.1, 48.9)
- added IC3: VNS3NV04DP-E, Package_SO:SO-8_3.9x4.9mm_P1.27mm, F.Cu at (58.4, 53.3)
- added IC4: VNS3NV04DP-E, Package_SO:SO-8_3.9x4.9mm_P1.27mm, F.Cu at (58.4, 62.2)
- added IC5: VNS3NV04DP-E, Package_SO:SO-8_3.9x4.9mm_P1.27mm, F.Cu at (58.4, 71.1)
- added R1: 180k, Resistor_SMD:R_0805_2012Metric, F.Cu at (172.5, 100.9)
- added R2: 180k, Resistor_SMD:R_0805_2012Metric, F.Cu at (184.2, 81.4)
- added R3: 330k, Resistor_SMD:R_0805_2012Metric, F.Cu at (184.2, 84.3)
- added R38: 100k, Resistor_SMD:R_0805_2012Metric, F.Cu at (65.7, 54.6)
- added R39: 100k, Resistor_SMD:R_0805_2012Metric, F.Cu at (69.5, 50.8)
- added R4: 330k, Resistor_SMD:R_0805_2012Metric, F.Cu at (184.2, 87.3)
- added R40: 100k, Resistor_SMD:R_0805_2012Metric, F.Cu at (70.2, 66.0)
- added R41: 100k, Resistor_SMD:R_0805_2012Metric, F.Cu at (65.7, 64.8)
- added R42: 100k, Resistor_SMD:R_0805_2012Metric, F.Cu at (69.5, 73.7)
- added R43: 100k, Resistor_SMD:R_0805_2012Metric, F.Cu at (68.9, 69.8)
- added R44: 1k, Resistor_SMD:R_0805_2012Metric, F.Cu at (69.5, 54.6)
- added R45: 1k, Resistor_SMD:R_0805_2012Metric, F.Cu at (65.1, 50.8)
- added R46: 1k, Resistor_SMD:R_0805_2012Metric, F.Cu at (69.5, 62.2)
- added R47: 1k, Resistor_SMD:R_0805_2012Metric, F.Cu at (65.7, 61.0)
- added R48: 1k, Resistor_SMD:R_0805_2012Metric, F.Cu at (65.7, 73.7)
- added R49: 1k, Resistor_SMD:R_0805_2012Metric, F.Cu at (65.7, 68.6)
- added R5: 330k, Resistor_SMD:R_0805_2012Metric, F.Cu at (184.2, 90.2)
- added R50: 680, Resistor_SMD:R_0805_2012Metric, F.Cu at (89.2, 53.3)
- added R51: 680, Resistor_SMD:R_0805_2012Metric, F.Cu at (88.9, 49.5)
- added R52: 680, Resistor_SMD:R_0805_2012Metric, F.Cu at (88.6, 62.2)
- added R53: 680, Resistor_SMD:R_0805_2012Metric, F.Cu at (88.6, 58.4)
- added R54: 680, Resistor_SMD:R_0805_2012Metric, F.Cu at (89.2, 72.4)
- added R55: 680, Resistor_SMD:R_0805_2012Metric, F.Cu at (89.2, 67.3)
- added R6: 330k, Resistor_SMD:R_0805_2012Metric, F.Cu at (176.9, 100.9)
- added R7: 180k, Resistor_SMD:R_0805_2012Metric, F.Cu at (184.2, 93.2)
- added R8: 180k, Resistor_SMD:R_0805_2012Metric, F.Cu at (184.2, 96.1)
- added R80: 100k, Resistor_SMD:R_0805_2012Metric, F.Cu at (209.0, 53.9)
- added R81: 100k, Resistor_SMD:R_0805_2012Metric, F.Cu at (213.4, 53.9)
- added R82: 1k, Resistor_SMD:R_0805_2012Metric, F.Cu at (217.9, 53.9)
- added R83: 1k, Resistor_SMD:R_0805_2012Metric, F.Cu at (222.3, 53.9)
- added R9: 10K, Resistor_SMD:R_0805_2012Metric, F.Cu at (141.8, -2.42)
- added U1: LMV324, Package_SO:SO-14_5.3x10.2mm_P1.27mm, F.Cu at (172.3, 82.0)
- C1, C10, C11, C12, C13, C14, C15, C16, C17, C18, C19, C2, C20, C21, C22, C23, C24, C25, C26, C27, C28, C3, C30, C31, C4, C5, C6, C7, C8, C9: footprint Capacitor_THT:CP_Radial_D5.0mm_P2.50mm -> Capacitor_SMD:C_0805_2012Metric
- C29: footprint Capacitor_THT:CP_Radial_D5.0mm_P2.50mm -> Capacitor_Tantalum_SMD:CP_EIA-7343-31_Kemet-D
- C32: footprint Capacitor_THT:CP_Radial_D5.0mm_P2.50mm -> Capacitor_Tantalum_SMD:CP_EIA-3528-21_Kemet-B
- D13, D14, D15, D16, D17, D18: footprint LED_THT:LED_D3.0mm -> LED_SMD:LED_0805_2012Metric
- D19: footprint Diode_THT:D_DO-41_SOD81_P10.16mm_Horizontal -> Diode_SMD:D_SMA
- D20: footprint Diode_THT:D_DO-35_SOD27_P10.16mm_Horizontal -> Diode_SMD:D_SMB
- D7: footprint Diode_THT:D_DO-41_SOD81_P10.16mm_Horizontal -> Diode_SMD:D_SOD-323
- IC1, IC2: footprint Connector_PinHeader_2.54mm:PinHeader_1x06_P2.54mm_Vertical -> Connector_PinHeader_2.54mm:PinHeader_1x05_P2.54mm_Vertical
- IC10, IC12: footprint Package_DIP:DIP-16_W7.62mm -> Package_SO:SOIC-16_3.9x9.9mm_P1.27mm
- IC6, IC7, IC8: footprint Package_DIP:DIP-10_W7.62mm -> Package_SO:SOIC-8_3.9x4.9mm_P1.27mm
- IC9: footprint Package_TO_SOT_THT:TO-3P-3_Vertical -> Package_TO_SOT_SMD:TO-263-3_TabPin2
- Q1, Q2, Q3: footprint Package_TO_SOT_THT:TO-3P-3_Vertical -> Package_TO_SOT_SMD:SOT-23
- R17, R18, R19, R20, R21, R22, R23, R24, R25, R26, R27, R28, R29, R30, R31, R32, R33, R34, R35, R36, R37, R56, R57, R58, R59, R60, R61, R62, R63, R64, R65, R66, R67, R68, R69, R70, R71, R72, R73, R74, R75, R76, R77, R78, R79, R92: footprint Resistor_THT:R_Axial_DIN0207_L6.3mm_D2.5mm_P2.54mm_Vertical -> Resistor_SMD:R_0805_2012Metric
- RV1: footprint Varistor:RV_Disc_D7mm_W5.7mm_P5mm -> Varistor:RV_Disc_D15.5mm_W4.7mm_P7.5mm
- Z1: footprint Diode_THT:D_DO-35_SOD27_P10.16mm_Horizontal -> Diode_SMD:D_SOD-323
- moved IC1 141.2 mm to (138.4, 21.6), turned to 270 degrees
- moved IC2 141.0 mm to (138.4, 16.5), turned to 270 degrees
- moved R17 121.0 mm to (171.7, 25.5)
- moved C4 120.0 mm to (170.2, 22.5)
- moved R20 114.1 mm to (169.1, 34.3)
- moved R19 113.7 mm to (160.2, 34.4)
- moved J5 113.2 mm to (210.1, 68.6), turned to 0 degrees
- moved R21 111.7 mm to (179.0, 22.5)
- moved JP5 110.9 mm to (87.6, 76.2), turned to 270 degrees
- moved J4 105.3 mm to (141.0, 137.2), turned to 90 degrees
- moved R68 101.4 mm to (65.7, 80.0)
- moved R69 99.5 mm to (65.7, 83.8)
- moved JP4 97.4 mm to (144.2, 31.1)
- moved JP3 92.7 mm to (147.5, 31.1)
- moved R63 86.9 mm to (51.7, 83.8)
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Connections:
- U3 pad 29: (no net) -> Reset

Commit message: VR Conditioner
Parts:
- moved C33 42.7 mm to (135.6, 36.8)
- moved R9 35.9 mm to (136.2, 33.0)
- moved D21 32.6 mm to (137.2, 27.9)
Connections:
- IC10 pad 5: (no net) -> ADCClamp08
- IC10 pad 9: ADCClamp08 -> (no net)
- IC12 pad 10: ADCClamp10 -> (no net)
- IC12 pad 11: ADCClamp11 -> (no net)
- IC12 pad 2: (no net) -> ADCClamp11
- IC12 pad 3: (no net) -> ADCClamp10
