File: reference/hardware/v0.3/Jag_Speedy/Jag_Speedy_VRConditioner/Jag_Speedy_VRConditioner.sch (KiCad schematic (older format))
At the start: 15 parts, among them IC1 MAX9926UAEE+, J1 Conn_02x04_Counter_Clockwise

Commit message: VR Cond PCB update
Parts:
- J1: value Conn_02x04_Counter_Clockwise -> Conn
Changed lines of the file:
@@
 P 3700 3850
 F 0 "J1" H 3750 4167 50  0000 C CNN
-F 1 "Conn_02x04_Counter_Clockwise" H 3750 4076 50  0000 C CNN
+F 1 "Conn" H 3750 4076 50  0000 C CNN
 F 2 "Connector_PinHeader_2.54mm:PinHeader_2x04_P2.54mm_Vertical" H 3700 3850 50  0001 C CNN
 F 3 "~" H 3700 3850 50  0001 C CNN

Commit message: VR PCB Update
Parts:
- R7, R8: footprint Resistor_SMD:R_0805_2012Metric -> Resistor_THT:R_Axial_DIN0414_L11.9mm_D4.5mm_P15.24mm_Horizontal
Changed lines of the file:
@@
 F 0 "R8" H 8350 4600 50  0000 C CNN
 F 1 "4.7K" H 8350 4700 50  0000 C CNN
-F 2 "Resistor_SMD:R_0805_2012Metric" V 8130 4650 50  0001 C CNN
+F 2 "Resistor_THT:R_Axial_DIN0414_L11.9mm_D4.5mm_P15.24mm_Horizontal" V 8130 4650 50  0001 C CNN
 F 3 "~" H 8200 4650 50  0001 C CNN
 	1    8200 4650
@@
 F 0 "R7" H 8300 3000 50  0000 C CNN
 F 1 "4.7K" H 8300 3100 50  0000 C CNN
-F 2 "Resistor_SMD:R_0805_2012Metric" V 8080 3050 50  0001 C CNN
+F 2 "Resistor_THT:R_Axial_DIN0414_L11.9mm_D4.5mm_P15.24mm_Horizontal" V 8080 3050 50  0001 C CNN
 F 3 "~" H 8150 3050 50  0001 C CNN
 	1    8150 3050

Commit message: PCB Changes
Parts:
- J1: footprint Connector_PinHeader_2.54mm:PinHeader_2x04_P2.54mm_Vertical -> Package_DIP:DIP-8_W7.62mm_Socket
Changed lines of the file:
@@
 F 0 "J1" H 3750 4167 50  0000 C CNN
 F 1 "Conn" H 3750 4076 50  0000 C CNN
-F 2 "Connector_PinHeader_2.54mm:PinHeader_2x04_P2.54mm_Vertical" H 3700 3850 50  0001 C CNN
+F 2 "Package_DIP:DIP-8_W7.62mm_Socket" H 3700 3850 50  0001 C CNN
 F 3 "~" H 3700 3850 50  0001 C CNN
 	1    3700 3850

Commit message: PCB Updates
Parts:
- R7: Component (none) -> Resistor
Changed lines of the file:
@@
 F 2 "Resistor_THT:R_Axial_DIN0414_L11.9mm_D4.5mm_P15.24mm_Horizontal" V 8080 3050 50  0001 C CNN
 F 3 "~" H 8150 3050 50  0001 C CNN
+F 4 "Resistor" H 8150 3050 50  0001 C CNN "Component"
 	1    8150 3050
 	-1   0    0    1

Commit message: PCB Changes
Parts:
- R7, R8: footprint Resistor_THT:R_Axial_DIN0414_L11.9mm_D4.5mm_P15.24mm_Horizontal -> Resistor_THT:R_Axial_DIN0411_L9.9mm_D3.6mm_P12.70mm_Horizontal
Changed lines of the file:
@@
 F 0 "R8" H 8350 4600 50  0000 C CNN
 F 1 "4.7K" H 8350 4700 50  0000 C CNN
-F 2 "Resistor_THT:R_Axial_DIN0414_L11.9mm_D4.5mm_P15.24mm_Horizontal" V 8130 4650 50  0001 C CNN
+F 2 "Resistor_THT:R_Axial_DIN0411_L9.9mm_D3.6mm_P12.70mm_Horizontal" V 8130 4650 50  0001 C CNN
 F 3 "~" H 8200 4650 50  0001 C CNN
 	1    8200 4650
@@
 F 0 "R7" H 8300 3000 50  0000 C CNN
 F 1 "4.7K" H 8300 3100 50  0000 C CNN
-F 2 "Resistor_THT:R_Axial_DIN0414_L11.9mm_D4.5mm_P15.24mm_Horizontal" V 8080 3050 50  0001 C CNN
+F 2 "Resistor_THT:R_Axial_DIN0411_L9.9mm_D3.6mm_P12.70mm_Horizontal" V 8080 3050 50  0001 C CNN
 F 3 "~" H 8150 3050 50  0001 C CNN
 F 4 "Resistor" H 8150 3050 50  0001 C CNN "Component"

Commit message: Tweaks
Parts:
- IC1: symbol MAX9926:MAX9926UAEE+ -> Jag_Speedy_VRConditioner-rescue:MAX9926UAEE+-MAX9926
Changed lines of the file:
@@
 $EndDescr
 $Comp
-L MAX9926:MAX9926UAEE+ IC1
+L Jag_Speedy_VRConditioner-rescue:MAX9926UAEE+-MAX9926 IC1
 U 1 1 5F034022
 P 5650 3650
