File: reference/hardware/Jag_Speedy/Jag_Speedy_VRConditioner/Jag_Speedy_VRConditioner.sch (KiCad schematic (older format))
At the start: 15 parts, among them IC1 MAX9926UAEE+, J1 Conn

Commit message: VR Gerbers & BOM
Parts:
- IC1: symbol MAX9926:MAX9926UAEE+ -> Jag_Speedy_VRConditioner-rescue:MAX9926UAEE+-MAX9926-Jag_Speedy_VRConditioner-rescue
Changed lines of the file:
@@
 $EndDescr
 $Comp
-L MAX9926:MAX9926UAEE+ IC1
+L Jag_Speedy_VRConditioner-rescue:MAX9926UAEE+-MAX9926-Jag_Speedy_VRConditioner-rescue IC1
 U 1 1 5F034022
 P 5650 3650
