File: reference/hardware/Jag_Speedy/inputs.sch (KiCad schematic (older format))
At the start: 51 parts, among them IC1 MPX4250AP, IC2 MPX4250AP, J6 Dual VR Conditioner

Commit message: EGR Input
Parts:
- added C34: 0.1uF, Capacitor_SMD:C_0805_2012Metric, symbol Device:C
- added C35: 0.22uF, Capacitor_SMD:C_0805_2012Metric, symbol Device:C
- added R12: 2.49k, Resistor_SMD:R_0805_2012Metric, symbol Device:R
- added R13: 470, Resistor_SMD:R_0805_2012Metric, symbol Device:R
Connections:
- net 3V3: now also R12.1
- net ADCClamp11: now also C35.1, R13.2
- net SensorGnd: now also C34.2, C35.2
- new net EGRSensor: C34.1, R12.2, R13.1
Other:
- note added: "Crank & Cam"
- note added: "Exhaust\nGas\nTemp"
Changed lines of the file:
@@
 Wire Wire Line
 	3100 5200 3300 5200
+Text Notes 8600 950  0    118  ~ 0
+Crank & Cam
+Text GLabel 9850 4500 2    50   Input ~ 0
+3V3
+Text GLabel 9850 5200 2    50   Input ~ 0
+SensorGnd
+Text GLabel 8500 4900 0    50   Input ~ 0
+EGRSensor
+$Comp
+L Device:R R13
+U 1 1 5F228D84
+P 9350 4900
+F 0 "R13" V 9557 4900 50  0000 C CNN
+F 1 "470" V 9466 4900 50  0000 C CNN
+F 2 "Resistor_SMD:R_0805_2012Metric" V 9280 4900 50  0001 C CNN
+F 3 "~" H 9350 4900 50  0001 C CNN
+	1    9350 4900
+	0    -1   -1   0
+$EndComp
+$Comp
+L Device:R R12
+U 1 1 5F228D8A
+P 8900 4650
+F 0 "R12" H 8970 4696 50  0000 L CNN
+F 1 "2.49k" H 8970 4605 50  0000 L CNN
+F 2 "Resistor_SMD:R_0805_2012Metric" V 8830 4650 50  0001 C CNN
+F 3 "~" H 8900 4650 50  0001 C CNN
+	1    8900 4650
+	1    0    0    -1
+$EndComp
+$Comp
+L Device:C C34
+U 1 1 5F228D90
+P 8900 5050
+F 0 "C34" H 9015 5096 50  0000 L CNN
+F 1 "0.1uF" H 9015 5005 50  0000 L CNN
+F 2 "Capacitor_SMD:C_0805_2012Metric" H 8938 4900 50  0001 C CNN
+F 3 "~" H 8900 5050 50  0001 C CNN
+	1    8900 5050
+	1    0    0    -1
+$EndComp
+$Comp
+L Device:C C35
+U 1 1 5F228D96
+P 9650 5050
+F 0 "C35" H 9765 5096 50  0000 L CNN
+F 1 "0.22uF" H 9765 5005 50  0000 L CNN
+F 2 "Capacitor_SMD:C_0805_2012Metric" H 9688 4900 50  0001 C CNN
+F 3 "~" H 9650 5050 50  0001 C CNN
+	1    9650 5050
+	1    0    0    -1
+$EndComp
+Wire Wire Line
+	9850 4500 8900 4500
+Wire Wire Line
+	8900 4800 8900 4900
+Wire Wire Line
+	8500 4900 8900 4900
+Connection ~ 8900 4900
+Wire Wire Line
+	9200 4900 8900 4900
+Wire Wire Line
+	9650 4900 9500 4900
+Connection ~ 9650 4900
+Wire Wire Line
+	9850 5200 9650 5200
+Wire Wire Line
+	9650 5200 8900 5200
+Connection ~ 9650 5200
+Text Notes 7950 4800 0    118  ~ 0
+Exhaust\nGas\nTemp
+Text GLabel 9850 4900 2    50   Output ~ 0
+EGR-Signal-3V3
+Wire Wire Line
+	9650 4900 9850 4900
+Text GLabel 9850 4800 2    50   Input ~ 0
+ADCClamp11
+Wire Wire Line
+	9850 4800 9650 4800
+Wire Wire Line
+	9650 4800 9650 4900
 $EndSCHEMATC
