File: reference/hardware/Jag_Speedy/EGT_Amp/EGT_Amp.sch (KiCad schematic (older format))
At the start: 17 parts, among them J1 Input, J2 Output, U1 AD8495, U2 AD8495, U3 AD8495

Commit message: final
Parts:
- J1, J2: footprint (none) -> Connector_PinHeader_2.54mm:PinHeader_1x04_P2.54mm_Vertical
Changed lines of the file:
@@
 F 0 "J1" H 3830 3392 50  0000 L CNN
 F 1 "Input" H 3830 3301 50  0000 L CNN
-F 2 "" H 3750 3400 50  0001 C CNN
+F 2 "Connector_PinHeader_2.54mm:PinHeader_1x04_P2.54mm_Vertical" H 3750 3400 50  0001 C CNN
 F 3 "~" H 3750 3400 50  0001 C CNN
 	1    3750 3400
@@
 F 0 "J2" H 3830 4292 50  0000 L CNN
 F 1 "Output" H 3830 4201 50  0000 L CNN
-F 2 "" H 3750 4250 50  0001 C CNN
+F 2 "Connector_PinHeader_2.54mm:PinHeader_1x04_P2.54mm_Vertical" H 3750 4250 50  0001 C CNN
 F 3 "~" H 3750 4250 50  0001 C CNN
 	1    3750 4250
